File: fpga.kicad_sch (KiCad schematic)
At the start: 0 parts

Commit message: stuff
Parts:
- added R17: R, symbol Device:R
Connections:
- new net DO.D6+: R17.1
Other:
- sheet FPGA pg.1 ports: added DO, FLASH_SPI; removed none
Changed lines of the file:
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@@
 	(generator_version "8.0")
 	(paper "A4")
+	(bus_entry
+		(at 99.06 36.83)
+		(size 2.54 2.54)
+		(stroke
+			(width 0)
+			(type default)
+		)
+	)
+	(wire
+		(pts
+			(xy 101.6 39.37) (xy 114.3 39.37)
+		)
+		(stroke
+			(width 0)
+			(type default)
+		)
+	)
+	(bus
+		(pts
+			(xy 91.44 76.2) (xy 99.06 76.2)
+		)
+		(stroke
+			(width 0)
+			(type default)
+		)
+	)
+	(bus
+		(pts
+			(xy 99.06 36.83) (xy 99.06 76.2)
+		)
+		(stroke
+			(width 0)
+			(type default)
+		)
+	)
+	(bus
+		(pts
+			(xy 99.06 34.29) (xy 99.06 36.83)
+		)
+		(stroke
+			(width 0)
+			(type default)
+		)
+	)
+	(label "DO.D6+"
+		(at 114.3 39.37 0)
+		(effects
+			(font
+				(size 1.27 1.27)
+			)
+			(justify left bottom)
+		)
+	)
+	(label "DO{D1+ D1- D2+ D2- D3+ D3- D4+ D4- D5+ D5- D6+ D6- D7+ D7- D8+ D8- D9+ D9- D10+ D10- D11+ D11- D12+ D12- D13+ D13- D14+ D14- D15+ D15- D16+ D16-}"
+		(at 92.71 76.2 0)
+		(fields_autoplaced yes)
+		(effects
+			(font
+				(size 1.27 1.27)
+			)
+			(justify left bottom)
+		)
+	)
+	(symbol
+		(lib_id "Device:R")
+		(at 114.3 43.18 0)
+		(unit 1)
+		(exclude_from_sim no)
+		(in_bom yes)
+		(on_board yes)
+		(dnp no)
+		(fields_autoplaced yes)
+		(property "Reference" "R17"
+			(at 116.84 41.9099 0)
+			(effects
+				(font
+					(size 1.27 1.27)
+				)
+				(justify left)
+			)
+		)
+		(property "Value" "R"
+			(at 116.84 44.4499 0)
+			(effects
+				(font
+					(size 1.27 1.27)
+				)
+				(justify left)
+			)
+		)
+		(property "Footprint" ""
+			(at 112.522 43.18 90)
+			(effects
+				(font
+					(size 1.27 1.27)
+				)
+				(hide yes)
+			)
+		)
+		(property "Datasheet" "~"
+			(at 114.3 43.18 0)
+			(effects
+				(font
+					(size 1.27 1.27)
+				)
+				(hide yes)
+			)
+		)
+		(property "Description" "Resistor"
+			(at 114.3 43.18 0)
+			(effects
+				(font
+					(size 1.27 1.27)
+				)
+				(hide yes)
+			)
+		)
+		(pin "2"
+		)
+		(pin "1"
+		)
+		(instances
+			(project "logix-core"
+				(path "/cf3b7c5f-6ddc-4e3f-9529-0bcf5eec6f23/824409ff-e0aa-4944-ad80-228eadb659f9"
+					(reference "R17")
+					(unit 1)
+				)
+			)
+		)
+	)
 	(sheet
 		(at 65.405 126.365)
@@
 	)
 	(sheet
-		(at 66.04 64.77)
-		(size 33.655 40.005)
+		(at 58.42 62.23)
+		(size 33.02 40.64)
 		(fields_autoplaced yes)
 		(stroke
@@
 		)
 		(property "Sheetname" "FPGA pg.1"
-			(at 66.04 64.0584 0)
+			(at 58.42 61.5184 0)
 			(effects
 				(font
@@
 		)
 		(property "Sheetfile" "fpga-pg1.kicad_sch"
-			(at 66.04 105.3596 0)
+			(at 58.42 103.4546 0)
 			(effects
 				(font
@@
 			)
 		)
+		(pin "FLASH_SPI" bidirectional
+			(at 91.44 85.725 0)
+			(effects
+				(font
+					(size 1.27 1.27)
+				)
+				(justify right)
+			)
+		)
+		(pin "DO" output
+			(at 91.44 76.2 0)
+			(effects
+				(font
+					(size 1.27 1.27)
+				)
+				(justify right)
+			)
+		)
