File: logix-core.kicad_pcb (KiCad board)
At the start: 6 copper layers, 62 parts, among them J1 QSH-030-01-X-D-A-XX, J2 QSH-030-01-X-D-A-XX, J3 878321420, U1 XC7A15T-FTG256, U2 MP5470GL-0000-P, U3 TPUSBLC6-4SC6, U4 FT230XQ, U5 MX25L3233FZN, U6 XC7A15T-CSG325

Commit message: working on ddr3
Parts:
- added C29: 100n, Capacitor_SMD:C_0402_1005Metric, F.Cu at (0.94, 7.46)
- added C30: 4.7u, Capacitor_SMD:C_0805_2012Metric, F.Cu at (201.7, 114.7)
- added C31: 100n, Capacitor_SMD:C_0603_1608Metric, F.Cu at (201.4, 104.4)
- added C32: 100n, Capacitor_SMD:C_0603_1608Metric, F.Cu at (201.4, 106.9)
- added C33: 100n, Capacitor_SMD:C_0603_1608Metric, F.Cu at (201.4, 109.4)
- added C34: 100n, Capacitor_SMD:C_0603_1608Metric, F.Cu at (201.4, 111.9)
- added C35: 4.7u, Capacitor_SMD:C_0805_2012Metric, F.Cu at (201.7, 117.7)
- added C36: 1u, Capacitor_SMD:C_0402_1005Metric, F.Cu at (192.5, 124.2)
- added C37: 1u, Capacitor_SMD:C_0402_1005Metric, F.Cu at (192.5, 126.1)
- added C38: 10n, Capacitor_SMD:C_0402_1005Metric, F.Cu at (192.5, 128.1)
- added C39: 10n, Capacitor_SMD:C_0402_1005Metric, F.Cu at (192.5, 130.1)
- added R17: 100, Capacitor_SMD:C_0402_1005Metric, F.Cu at (0.94, 3.50)
- added U1: XC7A15T-CSG325, Package_BGA:Xilinx_CSG325, F.Cu at (190.4, 112.1)
- added U8: MT41K256M16TW-107:P, MT41K256M16TW-107:FBGA96_8X14_MRN, F.Cu at (166.0, 143.5)
- moved C10 191.6 mm to (1.73, 1.00)
- moved U6 45.1 mm to (181.2, 142.8)
Connections:
- net VCCAUX renamed +V1P8
- C10 pad 1: VCCINT -> +V1P0
- C11 pad 1: VCCINT -> +V1P0
- C12 pad 1: VCCINT -> +V1P0
- C13 pad 1: VCCINT -> +V1P0
- C7 pad 1: VCCBRAM -> +V1P0
- C8 pad 1: VCCBRAM -> +V1P0
- C9 pad 1: VCCINT -> +V1P0
- J1 pad 01: /DI.DI2+ -> /Frontend Connector/DI.DI2+
- J1 pad 02: /DI.DI1+ -> /Frontend Connector/DI.DI1+
- J1 pad 03: /DI.DI2- -> /Frontend Connector/DI.DI2-
- J1 pad 04: /DI.DI1- -> /Frontend Connector/DI.DI1-
- J1 pad 05: /DI.DI3+ -> /Frontend Connector/DI.DI3+
- J1 pad 06: /DO.DO1+ -> /Frontend Connector/DO.DO1+
- J1 pad 07: /DI.DI3- -> /Frontend Connector/DI.DI3-
- J1 pad 08: /DO.DO1- -> /Frontend Connector/DO.DO1-
- J1 pad 09: /DI.DI4+ -> /Frontend Connector/DI.DI4+
- J1 pad 10: /DO.DO2+ -> /Frontend Connector/DO.DO2+
- J1 pad 11: /DI.DI4- -> /Frontend Connector/DI.DI4-
- J1 pad 12: /DO.DO2- -> /Frontend Connector/DO.DO2-
- J1 pad 13: /DI.DI5+ -> /Frontend Connector/DI.DI5+
- J1 pad 14: /DO.DO3+ -> /Frontend Connector/DO.DO3+
- J1 pad 15: /DI.DI5- -> /Frontend Connector/DI.DI5-
- J1 pad 16: /DO.DO3- -> /Frontend Connector/DO.DO3-
- J1 pad 17: /DI.DI6+ -> /Frontend Connector/DI.DI6+
- J1 pad 18: /DO.DO4+ -> /Frontend Connector/DO.DO4+
- J1 pad 19: /DI.DI6- -> /Frontend Connector/DI.DI6-
- J1 pad 20: /DO.DO4- -> /Frontend Connector/DO.DO4-
- J1 pad 21: /DI.DI7+ -> /Frontend Connector/DI.DI7+
- J1 pad 22: /DO.DO5+ -> /Frontend Connector/DO.DO5+
- J1 pad 23: /DI.DI7- -> /Frontend Connector/DI.DI7-
- J1 pad 24: /DO.DO5- -> /Frontend Connector/DO.DO5-
- J1 pad 25: /DI.DI8+ -> /Frontend Connector/DI.DI8+
- J1 pad 26: /DO.DO6+ -> /Frontend Connector/DO.DO6+
- J1 pad 27: /DI.DI8- -> /Frontend Connector/DI.DI8-
- J1 pad 28: /DO.DO6- -> /Frontend Connector/DO.DO6-
- J1 pad 29: /DI.DI9+ -> /Frontend Connector/DI.DI9+
- J1 pad 30: /DO.DO7+ -> /Frontend Connector/DO.DO7+
- J1 pad 31: /DI.DI9- -> /Frontend Connector/DI.DI9-
- J1 pad 32: /DO.DO7- -> /Frontend Connector/DO.DO7-
- J1 pad 33: /DI.DI10+ -> /Frontend Connector/DI.DI10+
- J1 pad 34: /DO.DO8+ -> /Frontend Connector/DO.DO8+
- J1 pad 35: /DI.DI10- -> /Frontend Connector/DI.DI10-
- J1 pad 36: /DO.DO8- -> /Frontend Connector/DO.DO8-
- J1 pad 37: /DI.DI11+ -> /Frontend Connector/DI.DI11+
- J1 pad 39: /DI.DI11- -> /Frontend Connector/DI.DI11-
- J1 pad 41: /DI.DI12+ -> /Frontend Connector/DI.DI12+
- J1 pad 43: /DI.DI12- -> /Frontend Connector/DI.DI12-
- J1 pad 45: /DI.DI13+ -> /Frontend Connector/DI.DI13+
- J1 pad 47: /DI.DI13- -> /Frontend Connector/DI.DI13-
- J1 pad 49: /DI.DI14+ -> /Frontend Connector/DI.DI14+
- J1 pad 51: /DI.DI14- -> /Frontend Connector/DI.DI14-
- J1 pad 53: /DI.DI15+ -> /Frontend Connector/DI.DI15+
- J1 pad 55: /DI.DI15- -> /Frontend Connector/DI.DI15-
- J1 pad 57: /DI.DI16+ -> /Frontend Connector/DI.DI16+
- J1 pad 59: /DI.DI16- -> /Frontend Connector/DI.DI16-
- U6 pad A2: unconnected-(U6D-MGTAVTT-PadA2) -> (no net)
- U6 pad A6: unconnected-(U6D-MGTRREF_216-PadA6) -> (no net)
- U6 pad B4: unconnected-(U6D-MGTAVCC-PadB4) -> (no net)
- U6 pad C1: unconnected-(U6D-MGTAVTT-PadC1) -> (no net)
- U6 pad C5: unconnected-(U6D-MGTAVCC-PadC5) -> (no net)
- U6 pad E1: unconnected-(U6D-MGTAVTT-PadE1) -> (no net)
- U6 pad E5: unconnected-(U6D-MGTAVCC-PadE5) -> (no net)
- U6 pad F11: VCCBRAM -> +V1P0
- U6 pad F3: unconnected-(U6D-MGTAVTT-PadF3) -> (no net)
- U6 pad F5: unconnected-(U6D-MGTAVCC-PadF5) -> (no net)
- U6 pad F7: VCCINT -> +V1P0
- U6 pad F9: VCCINT -> +V1P0
- U6 pad G10: VCCBRAM -> +V1P0
- U6 pad G2: unconnected-(U6D-MGTAVTT-PadG2) -> (no net)
- U6 pad G8: VCCINT -> +V1P0
- U6 pad H11: VCCBRAM -> +V1P0
- U6 pad H7: VCCINT -> +V1P0
- U6 pad H9: VCCINT -> +V1P0
- U6 pad J12: VCCINT -> +V1P0
- U6 pad J4: unconnected-(U6B-IO_L2N_T0_34-PadJ4) -> /DDR3_DQ4
- U6 pad J5: unconnected-(U6B-IO_L2P_T0_34-PadJ5) -> /DDR3_DQ3
- U6 pad J6: unconnected-(U6B-IO_0_34-PadJ6) -> /DDR3_DQ0
- U6 pad J8: VCCINT -> +V1P0
- U6 pad K1: unconnected-(U6B-IO_L3N_T0_DQS_34-PadK1) -> /DDR3_DQ6
- U6 pad K11: VCCINT -> +V1P0
- U6 pad K2: unconnected-(U6B-IO_L3P_T0_DQS_34-PadK2) -> /DDR3_DQ5
- U6 pad K3: unconnected-(U6B-IO_L4P_T0_34-PadK3) -> /DDR3_DQ7
- U6 pad K5: unconnected-(U6B-IO_L1N_T0_34-PadK5) -> /DDR3_DQ2
- U6 pad K6: unconnected-(U6B-IO_L1P_T0_34-PadK6) -> /DDR3_DQ1
- U6 pad K7: VCCINT -> +V1P0
- U6 pad L12: VCCINT -> +V1P0
- U6 pad L2: unconnected-(U6B-IO_L4N_T0_34-PadL2) -> /DDR3_DQ8
- U6 pad L3: unconnected-(U6B-IO_L5N_T0_34-PadL3) -> /DDR3_DQ10
- U6 pad L4: unconnected-(U6B-IO_L5P_T0_34-PadL4) -> /DDR3_DQ9
- U6 pad L5: unconnected-(U6B-IO_L6P_T0_34-PadL5) -> /DDR3_DQ11
- U6 pad L8: VCCINT -> +V1P0
- U6 pad M1: unconnected-(U6B-IO_L7N_T1_34-PadM1) -> /DDR3_DQ14
- U6 pad M11: VCCINT -> +V1P0
- U6 pad M2: unconnected-(U6B-IO_L7P_T1_34-PadM2) -> /DDR3_DQ13
- U6 pad M4: unconnected-(U6B-IO_L10P_T1_34-PadM4) -> /DDR3_ADDR3
- U6 pad M5: unconnected-(U6B-IO_L6N_T0_VREF_34-PadM5) -> /DDR3_DQ12
- U6 pad M6: unconnected-(U6B-IO_L8P_T1_34-PadM6) -> /DDR3_DQ15
- U6 pad M7: VCCINT -> +V1P0
- U6 pad N1: unconnected-(U6B-IO_L9P_T1_DQS_34-PadN1) -> /DDR3_ADDR1
- U6 pad N10: VCCINT -> +V1P0
- U6 pad N12: VCCINT -> +V1P0
- U6 pad N2: unconnected-(U6B-IO_L11N_T1_SRCC_34-PadN2) -> /DDR3_ADDR6
- U6 pad N3: unconnected-(U6B-IO_L11P_T1_SRCC_34-PadN3) -> /DDR3_ADDR5
- U6 pad N4: unconnected-(U6B-IO_L10N_T1_34-PadN4) -> /DDR3_ADDR4
- U6 pad N6: unconnected-(U6B-IO_L8N_T1_34-PadN6) -> /DDR3_ADDR0
- U6 pad N8: VCCINT -> +V1P0
- U6 pad P1: unconnected-(U6B-IO_L9N_T1_DQS_34-PadP1) -> /DDR3_ADDR2
- U6 pad P11: VCCINT -> +V1P0
- U6 pad P3: unconnected-(U6B-IO_L12N_T1_MRCC_34-PadP3) -> /DDR3_ADDR8
- U6 pad P4: unconnected-(U6B-IO_L12P_T1_MRCC_34-PadP4) -> /DDR3_ADDR7
- U6 pad P5: unconnected-(U6B-IO_L19N_T3_VREF_34-PadP5) -> /DDR3_BLOCK_ADDR2
- U6 pad P6: unconnected-(U6B-IO_L19P_T3_34-PadP6) -> /DDR3_BLOCK_ADDR1
- U6 pad P9: VCCINT -> +V1P0
- U6 pad R1: unconnected-(U6B-IO_L13N_T2_MRCC_34-PadR1) -> /DDR3_ADDR10
- U6 pad R2: unconnected-(U6B-IO_L13P_T2_MRCC_34-PadR2) -> /DDR3_ADDR9
- U6 pad R3: unconnected-(U6B-IO_L14P_T2_SRCC_34-PadR3) -> /DDR3_ADDR11
- U6 pad R5: unconnected-(U6B-IO_L21P_T3_DQS_34-PadR5) -> /DDR3_CLK_EN
- U6 pad R7: unconnected-(U6B-IO_L22P_T3_34-PadR7) -> /DDR3_ODT
- U6 pad T2: unconnected-(U6B-IO_L14N_T2_SRCC_34-PadT2) -> /DDR3_ADDR12
- U6 pad T3: unconnected-(U6B-IO_L17N_T2_34-PadT3) -> /DDR3_RESET#
- U6 pad T4: unconnected-(U6B-IO_L17P_T2_34-PadT4) -> /DDR3_RAS#
- U6 pad T5: unconnected-(U6B-IO_L21N_T3_DQS_34-PadT5) -> /DDR3_LDM
- U6 pad T7: unconnected-(U6B-IO_L22N_T3_34-PadT7) -> /DDR3_UDM
- U6 pad U1: unconnected-(U6B-IO_L15N_T2_DQS_34-PadU1) -> /DDR3_ADDR14
- U6 pad U2: unconnected-(U6B-IO_L15P_T2_DQS_34-PadU2) -> /DDR3_ADDR13
- U6 pad U4: unconnected-(U6B-IO_L18P_T2_34-PadU4) -> /DDR3_WE#
- U6 pad U5: unconnected-(U6B-IO_L20N_T3_34-PadU5) -> /DDR3_CLK-
- U6 pad U6: unconnected-(U6B-IO_L20P_T3_34-PadU6) -> /DDR3_CLK+
- U6 pad U7: unconnected-(U6B-IO_L23P_T3_34-PadU7) -> /DDR3_LDQS+
- U6 pad V2: unconnected-(U6B-IO_L16N_T2_34-PadV2) -> /DDR3_CS#
- U6 pad V3: unconnected-(U6B-IO_L16P_T2_34-PadV3) -> /DDR3_CAS#
- U6 pad V4: unconnected-(U6B-IO_L18N_T2_34-PadV4) -> /DDR3_BLOCK_ADDR0
- U6 pad V6: unconnected-(U6B-IO_L23N_T3_34-PadV6) -> /DDR3_LDQS-
- U6 pad V7: unconnected-(U6B-IO_L24N_T3_34-PadV7) -> /DDR3_UDQS-
- U6 pad V8: unconnected-(U6B-IO_L24P_T3_34-PadV8) -> /DDR3_UDQS+
Routing:
- net GND: track 21.2 -> 32.7 mm, vias 30 -> 51
- net +1V5: track 0.00 -> 9.85 mm, vias 0 -> 18
- net (no net): track 55.9 -> 61.5 mm, vias 79 -> 87
- net +V1P8: track 4.24 -> 0.00 mm, vias 6 -> 0
- net /DDR3_ADDR1: track 0.00 -> 3.33 mm, vias 0 -> 1
- net /DDR3_ADDR12: track 0.00 -> 3.24 mm, vias 0 -> 1
- net /DDR3_ADDR10: track 0.00 -> 3.01 mm, vias 0 -> 1
- net /DDR3_ADDR11: track 0.00 -> 2.97 mm, vias 0 -> 1
- net /DDR3_ADDR14: track 0.00 -> 2.53 mm, vias 0 -> 1
- net /DDR3_BLOCK_ADDR1: track 0.00 -> 2.45 mm, vias 0 -> 1
- net /DDR3_ADDR6: track 0.00 -> 2.01 mm, vias 0 -> 1
- net /DDR3_ADDR4: track 0.00 -> 1.97 mm, vias 0 -> 1
- net /DDR3_ADDR8: track 0.00 -> 1.97 mm, vias 0 -> 1
- net VCCBRAM: track 1.41 -> 0.00 mm, vias 2 -> 0
- net /DDR3/DDR_VREF: track 0.00 -> 1.14 mm, vias 0 -> 2
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
Commit message: working on ddr3 pcb
Routing:
- net GND: track 32.7 -> 80.7 mm, vias 51 -> 126
- net +V1P0: track 0.00 -> 11.9 mm, vias 0 -> 21
- net /DDR3_DQ6: track 0.57 -> 7.59 mm, vias 1 -> 2
- net /DDR3_LDQS-: track 0.57 -> 6.99 mm, vias 1 -> 2
- net /DDR3_LDQS+: track 0.52 -> 6.87 mm, vias 1 -> 3
- net /DDR3_DQ4: track 0.52 -> 6.54 mm, vias 1 -> 2
- net (no net): track 61.5 -> 67.2 mm, vias 87 -> 97
- net /DDR3_ADDR3: track 0.57 -> 6.05 mm, vias 1 -> 3
- net /DDR3_ADDR12: track 3.24 -> 8.57 mm, vias 1 -> 3
- net /DDR3_BLOCK_ADDR0: track 0.52 -> 5.49 mm, vias 1 -> 2
- net /DDR3_ADDR5: track 0.52 -> 5.49 mm, vias 1 -> 2
- net /DDR3_DQ13: track 0.57 -> 5.49 mm, vias 1 -> 2
- net /DDR3_DQ11: track 0.57 -> 5.49 mm, vias 1 -> 2
- net /DDR3_CS#: track 0.57 -> 5.49 mm, vias 1 -> 2
- net /DDR3_ADDR8: track 1.97 -> 6.88 mm, vias 1 -> 2
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
Commit message: working for ddr3 pcb part 2
Routing:
- net /DDR3_ADDR6: track 2.46 -> 15.7 mm
- net /DDR3_ADDR14: track 6.79 -> 19.9 mm
- net /DDR3_ADDR11: track 7.19 -> 20.2 mm
- net /DDR3_ADDR4: track 2.46 -> 14.7 mm
- net /DDR3_ADDR1: track 7.59 -> 19.5 mm
- net /DDR3_BLOCK_ADDR1: track 3.03 -> 14.1 mm
- net /DDR3/ZQ: track 1.89 -> 12.9 mm
- net /DDR3_ADDR10: track 5.78 -> 16.6 mm
- net /DDR3_ADDR8: track 6.88 -> 16.0 mm
- net GND: track 80.7 -> 75.4 mm
- net /DDR3_ADDR12: track 8.57 -> 13.5 mm
