File: logix-core.kicad_sch (KiCad schematic)
At the start: 0 parts

Commit message: stuff
Other:
- added sheet Backend Connector (backend_conn.kicad_sch)
- added sheet Frontend Connector (frontend_conn.kicad_sch)
- added sheet JTAG (jtag.kicad_sch)
- added sheet PMIC (pmic.kicad_sch)
Changed lines of the file:
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@@
 	(paper "A3")
+	(sheet
+		(at 322.58 146.05)
+		(size 36.83 44.45)
+		(fields_autoplaced yes)
+		(stroke
+			(width 0.1524)
+			(type solid)
+		)
+		(fill
+			(color 0 0 0 0.0000)
+		)
+		(property "Sheetname" "Frontend Connector"
+			(at 322.58 145.3384 0)
+			(effects
+				(font
+					(size 1.27 1.27)
+				)
+				(justify left bottom)
+			)
+		)
+		(property "Sheetfile" "frontend_conn.kicad_sch"
+			(at 322.58 191.0846 0)
+			(effects
+				(font
+					(size 1.27 1.27)
+				)
+				(justify left top)
+			)
+		)
+		(instances
+			(project "logix-core"
+				(path "/cf3b7c5f-6ddc-4e3f-9529-0bcf5eec6f23"
+					(page "7")
+				)
+			)
+		)
+	)
+	(sheet
+		(at 123.19 133.35)
+		(size 29.21 33.02)
+		(fields_autoplaced yes)
+		(stroke
+			(width 0.1524)
+			(type solid)
+		)
+		(fill
+			(color 0 0 0 0.0000)
+		)
+		(property "Sheetname" "PMIC"
+			(at 123.19 132.6384 0)
+			(effects
+				(font
+					(size 1.27 1.27)
+				)
+				(justify left bottom)
+			)
+		)
+		(property "Sheetfile" "pmic.kicad_sch"
+			(at 123.19 166.9546 0)
+			(effects
+				(font
+					(size 1.27 1.27)
+				)
+				(justify left top)
+			)
+		)
+		(instances
+			(project "logix-core"
+				(path "/cf3b7c5f-6ddc-4e3f-9529-0bcf5eec6f23"
+					(page "10")
+				)
+			)
+		)
+	)
+	(sheet
+		(at 200.66 92.71)
+		(size 34.29 39.37)
+		(fields_autoplaced yes)
+		(stroke
+			(width 0.1524)
+			(type solid)
+		)
+		(fill
+			(color 0 0 0 0.0000)
+		)
+		(property "Sheetname" "JTAG"
+			(at 200.66 91.9984 0)
+			(effects
+				(font
+					(size 1.27 1.27)
+				)
+				(justify left bottom)
+			)
+		)
+		(property "Sheetfile" "jtag.kicad_sch"
+			(at 200.66 132.6646 0)
+			(effects
+				(font
+					(size 1.27 1.27)
+				)
+				(justify left top)
+			)
+		)
+		(instances
+			(project "logix-core"
+				(path "/cf3b7c5f-6ddc-4e3f-9529-0bcf5eec6f23"
+					(page "9")
+				)
+			)
+		)
+	)
+	(sheet
+		(at 260.35 107.95)
+		(size 30.48 38.1)
+		(fields_autoplaced yes)
+		(stroke
+			(width 0.1524)
+			(type solid)
+		)
+		(fill
+			(color 0 0 0 0.0000)
+		)
+		(property "Sheetname" "Backend Connector"
+			(at 260.35 107.2384 0)
+			(effects
+				(font
+					(size 1.27 1.27)
+				)
+				(justify left bottom)
+			)
+		)
+		(property "Sheetfile" "backend_conn.kicad_sch"
+			(at 260.35 146.6346 0)
+			(effects
+				(font
+					(size 1.27 1.27)
+				)
+				(justify left top)
+			)
+		)
+		(instances
+			(project "logix-core"
+				(path "/cf3b7c5f-6ddc-4e3f-9529-0bcf5eec6f23"
+					(page "8")
+				)
+			)
+		)
+	)
 	(sheet
 		(at 184.15 188.595)

Commit message: more stuff!
Other:
- added sheet SPI Flash (spi_flash.kicad_sch)
- added sheet USB (usb.kicad_sch)
Changed lines of the file:
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@@
+	)
+	(sheet
+		(at 95.25 59.69)
+		(size 31.75 35.56)
+		(fields_autoplaced yes)
+		(stroke
+			(width 0.1524)
+			(type solid)
+		)
+		(fill
+			(color 0 0 0 0.0000)
+		)
+		(property "Sheetname" "USB"
+			(at 95.25 58.9784 0)
+			(effects
+				(font
+					(size 1.27 1.27)
+				)
+				(justify left bottom)
+			)
+		)
+		(property "Sheetfile" "usb.kicad_sch"
+			(at 95.25 95.8346 0)
+			(effects
+				(font
+					(size 1.27 1.27)
+				)
+				(justify left top)
+			)
+		)
+		(instances
+			(project "logix-core"
+				(path "/cf3b7c5f-6ddc-4e3f-9529-0bcf5eec6f23"
+					(page "11")
+				)
+			)
+		)
 	)
 	(sheet
@@
 				)
 			)
+		)
+	)
+	(sheet
+		(at 54.61 182.88)
+		(size 34.29 41.91)
+		(fields_autoplaced yes)
+		(stroke
+			(width 0.1524)
+			(type solid)
+		)
+		(fill
+			(color 0 0 0 0.0000)
+		)
+		(property "Sheetname" "SPI Flash"
+			(at 54.61 182.1684 0)
+			(effects
+				(font
+					(size 1.27 1.27)
+				)
+				(justify left bottom)
+			)
+		)
+		(property "Sheetfile" "spi_flash.kicad_sch"
+			(at 54.61 225.3746 0)
+			(effects
+				(font
+					(size 1.27 1.27)
+				)
+				(justify left top)
+			)
+		)
+		(instances
+			(project "logix-core"
+				(path "/cf3b7c5f-6ddc-4e3f-9529-0bcf5eec6f23"
+					(page "12")
+				)
+			)

Commit message: stuff
Other:
- sheet FPGA ports: added DI, DO; removed none
- sheet Frontend Connector ports: added DI, DO; removed none
Changed lines of the file:
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@@
 	(generator_version "8.0")
 	(paper "A3")
-	(sheet
-		(at 322.58 146.05)
+	(bus
+		(pts
+			(xy 241.3 196.85) (xy 287.02 196.85)
+		)
+		(stroke
+			(width 0)
+			(type default)
+		)
+	)
+	(bus
+		(pts
+			(xy 241.3 199.39) (xy 287.02 199.39)
+		)
+		(stroke
+			(width 0)
+			(type default)
+		)
+	)
+	(label "DI{DI1+ DI1- DI2+ DI2- DI3+ DI3- DI4+ DI4- DI5+ DI5- DI6+ DI6- DI7+ DI7- DI8+ DI8- DI9+ DI9- DI10+ DI10- DI11+ DI11- DI12+ DI12- DI13+ DI13- DI14+ DI14- DI15+ DI15- DI16+ DI16-}"
+		(at 242.57 199.39 0)
+		(fields_autoplaced yes)
+		(effects
+			(font
+				(size 1.27 1.27)
+			)
+			(justify left bottom)
+		)
+	)
+	(label "DO{DO1+ DO1- DO2+ DO2- DO3+ DO3- DO4+ DO4- DO5+ DO5- DO6+ DO6- DO7+ DO7- DO8+ DO8-}"
+		(at 242.57 196.85 0)
+		(fields_autoplaced yes)
+		(effects
+			(font
+				(size 1.27 1.27)
+			)
+			(justify left bottom)
+		)
+	)
+	(sheet
+		(at 287.02 187.96)
 		(size 36.83 44.45)
 		(fields_autoplaced yes)
@@
 		)
 		(property "Sheetname" "Frontend Connector"
-			(at 322.58 145.3384 0)
+			(at 287.02 187.2484 0)
 			(effects
 				(font
@@
 		)
 		(property "Sheetfile" "frontend_conn.kicad_sch"
-			(at 322.58 191.0846 0)
-			(effects
-				(font
-					(size 1.27 1.27)
-				)
-				(justify left top)
+			(at 287.02 232.9946 0)
+			(effects
+				(font
+					(size 1.27 1.27)
+				)
+				(justify left top)
+			)
+		)
+		(pin "DI" output
+			(at 287.02 199.39 180)
+			(effects
+				(font
+					(size 1.27 1.27)
+				)
+				(justify left)
+			)
+		)
+		(pin "DO" input
+			(at 287.02 196.85 180)
+			(effects
+				(font
+					(size 1.27 1.27)
+				)
+				(justify left)
 			)
 		)
@@
 	(sheet
 		(at 184.15 188.595)
-		(size 56.515 64.77)
+		(size 57.15 64.77)
 		(fields_autoplaced yes)
 		(stroke
@@
 			)
 		)
+		(pin "DO" output
+			(at 241.3 196.85 0)
+			(effects
+				(font
+					(size 1.27 1.27)
+				)
+				(justify right)
+			)
+		)
+		(pin "DI" input
+			(at 241.3 199.39 0)
+			(effects
+				(font
+					(size 1.27 1.27)
+				)
+				(justify right)
+			)
+		)

Commit message: working on ddr3
Other:
- added sheet DDR3 (ddr3.kicad_sch)
- sheet FPGA ports: added DDR3_ADDR, DDR3_BLOCK_ADDR, DDR3_CAS#, DDR3_CLK+, DDR3_CLK-, DDR3_CLK_EN, DDR3_CS#, DDR3_DQ, DDR3_LDM, DDR3_LDQS+, DDR3_LDQS-, DDR3_ODT, DDR3_RAS#, DDR3_RESET#, DDR3_UDM, DDR3_UDQS+, DDR3_UDQS-, DDR3_WE#; removed none
