File: _autosave-logix-core.kicad_sch (KiCad schematic)
At the start: 0 parts

Commit message: more ddr3, rules and stuff
Changed lines of the file:
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@@
 	(generator_version "9.0")
 	(paper "A3")
-	(junction
-		(at 191.77 143.51)
-		(diameter 0)
-		(color 0 0 0 0)
-	)
 	(wire
 		(pts
@@
 		)
 	)
+	(wire
+		(pts
+			(xy 189.23 171.45) (xy 233.68 171.45)
+		)
+		(stroke
+			(width 0)
+			(type default)
+		)
+	)
 	(bus
 		(pts
-			(xy 191.77 143.51) (xy 189.23 143.51)
-		)
-		(stroke
-			(width 0)
-			(type default)
-		)
-	)
-	(wire
-		(pts
-			(xy 189.23 171.45) (xy 233.68 171.45)
+			(xy 189.23 143.51) (xy 233.68 143.51)
+		)
+		(stroke
+			(width 0)
+			(type default)
+		)
+	)
+	(wire
+		(pts
+			(xy 189.23 176.53) (xy 233.68 176.53)
 		)
 		(stroke
@@
 	(bus
 		(pts
-			(xy 191.77 143.51) (xy 233.68 143.51)
-		)
-		(stroke
-			(width 0)
-			(type default)
-		)
-	)
-	(wire
-		(pts
-			(xy 189.23 176.53) (xy 233.68 176.53)
+			(xy 187.96 123.825) (xy 233.68 123.825)
+		)
+		(stroke
+			(width 0)
+			(type default)
+		)
+	)
+	(wire
+		(pts
+			(xy 189.23 191.77) (xy 233.68 191.77)
+		)
+		(stroke
+			(width 0)
+			(type default)
+		)
+	)
+	(wire
+		(pts
+			(xy 189.23 182.88) (xy 233.68 182.88)
 		)
 		(stroke
@@
 	(bus
 		(pts
-			(xy 187.96 123.825) (xy 233.68 123.825)
-		)
-		(stroke
-			(width 0)
-			(type default)
-		)
-	)
-	(wire
-		(pts
-			(xy 189.23 191.77) (xy 233.68 191.77)
-		)
-		(stroke
-			(width 0)
-			(type default)
-		)
-	)
-	(wire
-		(pts
-			(xy 189.23 182.88) (xy 233.68 182.88)
+			(xy 187.96 126.365) (xy 233.68 126.365)
 		)
 		(stroke
@@
 	(bus
 		(pts
-			(xy 187.96 126.365) (xy 233.68 126.365)
-		)
-		(stroke
-			(width 0)
-			(type default)
-		)
-	)
-	(bus
-		(pts
 			(xy 189.23 167.64) (xy 233.68 167.64)
 		)
@@
 		(pts
 			(xy 189.23 173.99) (xy 233.68 173.99)
-		)
-		(stroke
-			(width 0)
-			(type default)
-		)
-	)
-	(bus
-		(pts
-			(xy 191.77 142.24) (xy 191.77 143.51)
 		)
 		(stroke
@@
 			(effects
 				(font
-					(size 1.27 1.27)
-					(italic yes)
-				)
-			)
-		)
-	)
-	(netclass_flag ""
-		(length 7)
-		(shape round)
-		(at 191.77 142.24 0)
-		(fields_autoplaced yes)
-		(effects
-			(font
-				(size 1.27 1.27)
-			)
-			(justify left bottom)
-		)
-		(property "Netclass" "DDR3_DQ"
-			(at 192.4685 135.24 0)
-			(effects
-				(font
-					(size 1.27 1.27)
-				)
-				(justify left)
-			)
-		)
-		(property "Component Class" ""
-			(at -152.4 15.24 0)
-			(effects
-				(font
