File: 7-segment.kicad_sch (KiCad schematic)
At the start: 0 parts

Commit message: added a lot of stuff
Parts:
- added LED1: SLS0391FR1A1GD_C2913076, SLS0391FR1A1GD:LED-SEG-SMD_10P-L13.0-W9.8-P1.88-S13.70-BL, symbol SLS0391FR1A1GD:SLS0391FR1A1GD_C2913076
- added Q1: TPNTK3139PT1G, TPNTK3139PT1G:SOT-723_L1.2-W0.8-P0.40-LS1.2-BR, symbol TPNTK3139PT1G:TPNTK3139PT1G
- added Q2, Q3, Q4, Q5, Q6, Q7, Q8, Q9: 2N7002M3T5G-ES, 2N7002M3T5G-ES:SOT-723_L1.2-W0.8-P0.80-LS1.2-BL, symbol 2N7002M3T5G-ES:2N7002M3T5G-ES
- added R21, R30, R31, R32, R33, R34, R35, R36, R37: 100k, Resistor_SMD:R_0402_1005Metric, symbol Device:R
- added R22, R23, R24, R25, R26, R27, R28, R29: 68, Resistor_SMD:R_0402_1005Metric, symbol Device:R
- added R72: 0, Resistor_SMD:R_0402_1005Metric, symbol Device:R
Connections:
- new net: Q1.2 (S), R21.1, R72.2
- new net +3.3V: R72.1
- new net 7SEG_A: Q1.1 (G), R21.2
- new net 7SEG_A_DRAIN: LED1.3 (COM), LED1.8 (COM), Q1.3 (D)
- new net 7SEG_C0: Q2.1 (G), R30.1
- new net 7SEG_C1: Q3.1 (G), R31.1
- new net 7SEG_C2: Q4.1 (G), R32.1
- new net 7SEG_C3: Q5.1 (G), R33.1
- new net 7SEG_C4: Q6.1 (G), R34.1
- new net 7SEG_C5: Q7.1 (G), R35.1
- new net 7SEG_C6: Q8.1 (G), R36.1
- new net 7SEG_C7: Q9.1 (G), R37.1
- new net 7SEG_CA: LED1.7 (A), R22.2
- new net 7SEG_CA_DRAIN: Q2.3 (D), R22.1
- new net 7SEG_CB: LED1.6 (B), R23.2
- new net 7SEG_CB_DRAIN: Q3.3 (D), R23.1
- new net 7SEG_CC: LED1.4 (C), R24.2
- new net 7SEG_CC_DRAIN: Q4.3 (D), R24.1
- new net 7SEG_CD: LED1.2 (D), R25.2
- new net 7SEG_CDP: LED1.5 (DP), R29.2
- new net 7SEG_CDP_DRAIN: Q9.3 (D), R29.1
- new net 7SEG_CD_DRAIN: Q5.3 (D), R25.1
- new net 7SEG_CE: LED1.1 (E), R26.2
- new net 7SEG_CE_DRAIN: Q6.3 (D), R26.1
- new net 7SEG_CF: LED1.9 (F), R27.2
- new net 7SEG_CF_DRAIN: Q7.3 (D), R27.1
- new net 7SEG_CG: LED1.10 (G), R28.2
- new net 7SEG_CG_DRAIN: Q8.3 (D), R28.1
- new net GND: Q2.2 (S), Q3.2 (S), Q4.2 (S), Q5.2 (S), Q6.2 (S), Q7.2 (S), Q8.2 (S), Q9.2 (S), R30.2, R31.2, R32.2, R33.2, R34.2, R35.2, R36.2, R37.2

Commit message: did alot of stuff
Parts:
- LED1: LCSC (none) -> C2913076
- Q1: LCSC (none) -> C558623
- Q2, Q3, Q4, Q5, Q6, Q7, Q8, Q9: LCSC (none) -> C5224234
- R21, R30, R31, R32, R33, R34, R35, R36, R37: LCSC (none) -> C25741
- R22, R23, R24, R25, R26, R27, R28, R29: LCSC (none) -> C163455
- R72: LCSC (none) -> C17168
Changed lines of the file:
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@@
 			)
 		)
+		(property "LCSC" "C25741"
+			(at 97.79 152.4 0)
+			(effects
+				(font
+					(size 1.27 1.27)
+				)
+			)
+		)
 		(pin "1"
 		)
@@
 			)
 		)
+		(property "LCSC" "C5224234"
+			(at 125.73 100.33 0)
+			(effects
+				(font
+					(size 1.27 1.27)
+				)
+			)
+		)
 		(pin "1"
 		)
@@
 			)
 		)
+		(property "LCSC" "C25741"
+			(at 128.27 152.4 0)
+			(effects
+				(font
+					(size 1.27 1.27)
+				)
+			)
+		)
 		(pin "1"
 		)
@@
 			)
 		)
+		(property "LCSC" "C25741"
+			(at 143.51 39.37 0)
+			(effects
+				(font
+					(size 1.27 1.27)
+				)
+			)
+		)
 		(pin "1"
 		)
@@
 			)
 		)
+		(property "LCSC" "C163455"
+			(at 198.12 109.22 0)
+			(effects
+				(font
+					(size 1.27 1.27)
+				)
+			)
+		)
 		(pin "2"
 		)
@@
 			)
 		)
+		(property "LCSC" "C5224234"
+			(at 147.32 140.97 0)
+			(effects
+				(font
+					(size 1.27 1.27)
+				)
+			)
+		)
 		(pin "1"
 		)
@@
 			)
 		)
+		(property "LCSC" "C17168"
+			(at 161.29 27.94 0)
+			(effects
+				(font
+					(size 1.27 1.27)
+				)
+			)
+		)
 		(pin "1"
 		)
@@
 			)
 		)
+		(property "LCSC" "C25741"
+			(at 120.65 152.4 0)
+			(effects
+				(font
+					(size 1.27 1.27)
+				)
+			)
+		)
 		(pin "1"
 		)
@@
 			)
 		)
+		(property "LCSC" "C163455"
+			(at 198.12 99.06 0)
+			(effects
+				(font
+					(size 1.27 1.27)
+				)
+			)
+		)
 		(pin "2"
 		)
@@
 			)
 		)
+		(property "LCSC" "C5224234"
+			(at 135.89 120.65 0)
+			(effects
+				(font
+					(size 1.27 1.27)
+				)
+			)
+		)
 		(pin "1"
 		)
@@
 			)
 		)
+		(property "LCSC" "C5224234"
+			(at 114.3 80.01 0)
+			(effects
+				(font
+					(size 1.27 1.27)
+				)
+			)
+		)
 		(pin "1"
 		)
@@
 			)
 		)
+		(property "LCSC" "C5224234"
+			(at 119.38 90.17 0)
+			(effects
+				(font
+					(size 1.27 1.27)
+				)
+			)
+		)
 		(pin "1"
 		)
@@
 			)
 		)
+		(property "LCSC" "C163455"
+			(at 198.12 101.6 0)
+			(effects
+				(font
+					(size 1.27 1.27)
+				)
+			)
+		)
 		(pin "2"
 		)
@@
 			)
 		)
+		(property "LCSC" "C163455"
+			(at 198.12 96.52 0)
+			(effects
+				(font
+					(size 1.27 1.27)
+				)
+			)
+		)
 		(pin "2"
 		)
@@
 			)
 		)
+		(property "LCSC" "C163455"
+			(at 198.12 106.68 0)
+			(effects
+				(font
+					(size 1.27 1.27)
+				)
+			)
+		)
 		(pin "2"
 		)
@@
 			)
 		)
+		(property "LCSC" "C5224234"
+			(at 142.24 130.81 0)
+			(effects
+				(font
+					(size 1.27 1.27)
+				)
+			)
+		)
 		(pin "1"
 		)
@@
 			)
 		)
+		(property "LCSC" "C558623"
+			(at 161.29 48.26 0)
+			(effects
+				(font
+					(size 1.27 1.27)
+				)
+			)
+		)
 		(pin "1"
 		)
@@
 			)
 		)
+		(property "LCSC" "C5224234"
+			(at 130.81 110.49 0)
+			(effects
+				(font
+					(size 1.27 1.27)
+				)
+			)
+		)
 		(pin "1"
 		)
@@
 			)
 		)
+		(property "LCSC" "C163455"
+			(at 198.12 104.14 0)
+			(effects
+				(font
+					(size 1.27 1.27)
+				)
+			)
+		)
 		(pin "2"
 		)
@@
 			)
 		)
+		(property "LCSC" "C25741"
+			(at 105.41 152.4 0)
+			(effects
+				(font
+					(size 1.27 1.27)
+				)
+			)
+		)
 		(pin "1"
 		)
@@
 			)
 		)
+		(property "LCSC" "C25741"
+			(at 113.03 152.4 0)
+			(effects
+				(font
+					(size 1.27 1.27)
+				)
+			)
+		)
 		(pin "1"
 		)
@@
 			)
 		)
+		(property "LCSC" "C25741"
+			(at 135.89 152.4 0)
+			(effects
+				(font
+					(size 1.27 1.27)
+				)
+			)
+		)
 		(pin "1"
 		)
@@
 			)
 		)
+		(property "LCSC" "C2913076"
+			(at 236.22 100.33 0)
+			(effects
+				(font
+					(size 1.27 1.27)
+				)
+			)
+		)
 		(pin "8"
 		)
@@
 			)
 		)
+		(property "LCSC" "C5224234"
+			(at 109.22 69.85 0)
+			(effects
+				(font
+					(size 1.27 1.27)
+				)
+			)
+		)
 		(pin "1"
 		)
@@
 			)
 		)
+		(property "LCSC" "C25741"
+			(at 90.17 152.4 0)
+			(effects
+				(font
+					(size 1.27 1.27)
+				)
+			)
+		)
 		(pin "1"
 		)
@@
 			)
 		)
+		(property "LCSC" "C25741"
+			(at 82.55 152.4 0)
+			(effects
+				(font
+					(size 1.27 1.27)
+				)
+			)
+		)
 		(pin "1"
 		)
@@
 			)
 		)
+		(property "LCSC" "C163455"
+			(at 198.12 91.44 0)
+			(effects
+				(font
+					(size 1.27 1.27)
+				)
+			)
+		)
 		(pin "2"
 		)
@@
 			)
 		)
+		(property "LCSC" "C163455"
+			(at 198.12 93.98 0)
+			(effects
+				(font
+					(size 1.27 1.27)
+				)
+			)
+		)
