File: fpga-pg1.kicad_sch (KiCad schematic)
At the start: 63 parts, among them U1 XC7A35T-FGG484

Commit message: filled out back connector, finished ddr pinning according to vivado
Parts:
- removed TP17, TP18, TP19, TP20, TP21, TP22, TP23, TP24, TP25, TP26, TP27, TP28, TP29, TP30, TP31, TP32, TP49, TP50, TP51, TP52, TP53, TP54, TP55, TP56, TP57, TP58, TP59, TP60, TP61, TP62, TP63, TP64, TP65, TP66, TP67, TP68, TP69, TP70, TP71, TP72, TP73, TP74, TP75, TP76, TP77, TP78, TP79, TP80: TestPoint_Small, symbol Connector:TestPoint_Small
Connections:
- net SYSRST#: now reaches U1.N15 (IO_25_14)
- net SYSCLK: now reaches U1.U20 (IO_L11P_T1_SRCC_14)

Commit message: added a lot of stuff
Parts:
- renumbered C43 to C1, C52 to C10, C51 to C11, C50 to C12, C49 to C13, C64 to C14, C44 to C2, C45 to C3, C46 to C4, C47 to C5, C48 to C6, C60 to C7, C61 to C8, C53 to C9
Connections:
- net DIP_SW2: now reaches U1.AA18 (IO_L17P_T2_A14_D30_14)
- net 7SEG3_C6: now reaches U1.AA19 (IO_L15P_T2_DQS_RDWR_B_14)
- net 7SEG2_C5: now reaches U1.AA20 (IO_L8P_T1_D11_14)
- net 7SEG2_C6: now reaches U1.AA21 (IO_L8N_T1_D12_14)
- net DIP_SW3: now reaches U1.AB18 (IO_L17N_T2_A13_D29_14)
- net 7SEG3_C7: now reaches U1.AB20 (IO_L15N_T2_DQS_DOUT_CSO_B_14)
- net BTN2#: now reaches U1.AB21 (IO_L10P_T1_D14_14)
- net 7SEG2_A: now reaches U1.P19 (IO_L5P_T0_D06_14)
- net 7SEG1_A: now reaches U1.P20 (IO_0_14)
- net 7SEG1_C2: now reaches U1.P21 (IO_L2P_T0_D02_14)
- net 7SEG1_C0: now reaches U1.P22 (IO_L1P_T0_D00_MOSI_14)
- net 7SEG2_C0: now reaches U1.R19 (IO_L5N_T0_D07_14)
- net 7SEG1_C3: now reaches U1.R21 (IO_L2N_T0_D03_14)
- net 7SEG1_C1: now reaches U1.R22 (IO_L1N_T0_D01_DIN_14)
- net 7SEG2_C1: now reaches U1.T19 (IO_L6P_T0_FCS_B_14)
- net 7SEG2_C2: now reaches U1.T20 (IO_L6N_T0_D08_VREF_14)
- net 7SEG1_C6: now reaches U1.T21 (IO_L4P_T0_D04_14)
- net 7SEG1_C7: now reaches U1.U21 (IO_L4N_T0_D05_14)
- net 7SEG1_C4: now reaches U1.U22 (IO_L3P_T0_DQS_PUDC_B_14)
- net DIP_SW0: now reaches U1.V17 (IO_L16P_T2_CSI_B_14)
- net 7SEG3_C4: now reaches U1.V18 (IO_L14P_T2_SRCC_14)
- net 7SEG3_C5: now reaches U1.V19 (IO_L14N_T2_SRCC_14)
- net 7SEG3_A: now reaches U1.V20 (IO_L11N_T1_SRCC_14)
- net 7SEG1_C5: now reaches U1.V22 (IO_L3N_T0_DQS_EMCCLK_14)
- net DIP_SW1: now reaches U1.W17 (IO_L16N_T2_A15_D31_14)
- net 7SEG3_C0: now reaches U1.W19 (IO_L12P_T1_MRCC_14)
- net 7SEG3_C1: now reaches U1.W20 (IO_L12N_T1_MRCC_14)
- net 7SEG2_C3: now reaches U1.W21 (IO_L7P_T1_D09_14)
- net 7SEG2_C4: now reaches U1.W22 (IO_L7N_T1_D10_14)
- net 7SEG3_C2: now reaches U1.Y18 (IO_L13P_T2_MRCC_14)
- net 7SEG3_C3: now reaches U1.Y19 (IO_L13N_T2_MRCC_14)
- net 7SEG2_C7: now reaches U1.Y21 (IO_L9P_T1_DQS_14)
- net BTN1#: now reaches U1.Y22 (IO_L9N_T1_DQS_D13_14)
- net SYSRST# renamed RST_BTN#

Commit message: did alot of stuff
Parts:
- C1, C14: footprint Capacitor_SMD:C_1210_3225Metric -> Capacitor_SMD:C_1206_3216Metric; LCSC (none) -> C96123
- C10, C11, C4, C5, C6, C7, C8, C9: LCSC (none) -> C47339
- C12, C13, C2, C3: LCSC (none) -> C23733
- U1: LCSC (none) -> C1521727
Changed lines of the file:
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@@
+			)
+		)
+		(property "LCSC" "C23733"
+			(at 97.79 62.23 0)
+			(effects
+				(font
+					(size 1.27 1.27)
+				)
 			)
 		)
@@
 			)
 		)
+		(property "LCSC" "C47339"
+			(at 254 62.23 0)
+			(effects
+				(font
+					(size 1.27 1.27)
+				)
+			)
+		)
 		(pin "2"
 		)
@@
 				)
 				(hide yes)
+			)
+		)
+		(property "LCSC" "C23733"
+			(at 317.5 62.23 0)
+			(effects
+				(font
+					(size 1.27 1.27)
+				)
 			)
 		)
@@
 			)
 		)
+		(property "LCSC" "C47339"
+			(at 292.1 62.23 0)
+			(effects
+				(font
+					(size 1.27 1.27)
+				)
+			)
+		)
 		(pin "2"
 		)
@@
 				)
 				(hide yes)
+			)
+		)
+		(property "LCSC" "C47339"
+			(at 110.49 62.23 0)
+			(effects
+				(font
+					(size 1.27 1.27)
+				)
 			)
 		)
@@
 			)
 		)
+		(property "LCSC" "C47339"
+			(at 135.89 62.23 0)
+			(effects
+				(font
+					(size 1.27 1.27)
+				)
+			)
+		)
 		(pin "2"
 		)
@@
 			)
 		)
-		(property "Footprint" "Capacitor_SMD:C_1210_3225Metric"
+		(property "Footprint" "Capacitor_SMD:C_1206_3216Metric"
 			(at 73.3552 66.04 0)
 			(effects
@@
 				)
 				(hide yes)
+			)
+		)
+		(property "LCSC" "C96123"
+			(at 72.39 62.23 0)
+			(effects
+				(font
+					(size 1.27 1.27)
+				)
 			)
 		)
@@
 				)
 				(hide yes)
+			)
+		)
+		(property "LCSC" "C47339"
+			(at 148.59 62.23 0)
+			(effects
+				(font
+					(size 1.27 1.27)
+				)
 			)
 		)
@@
 			)
 		)
+		(property "LCSC" "C47339"
+			(at 266.7 62.23 0)
+			(effects
+				(font
+					(size 1.27 1.27)
+				)
+			)
+		)
 		(pin "2"
 		)
@@
 			)
 		)
+		(property "LCSC" "C23733"
+			(at 85.09 62.23 0)
+			(effects
+				(font
+					(size 1.27 1.27)
+				)
+			)
+		)
 		(pin "2"
 		)
@@
 			)
 		)
+		(property "LCSC" "C23733"
+			(at 304.8 62.23 0)
+			(effects
+				(font
+					(size 1.27 1.27)
+				)
+			)
+		)
 		(pin "2"
 		)
@@
 			)
 		)
+		(property "LCSC" "C1521727"
+			(at 201.93 148.59 0)
+			(effects
+				(font
+					(size 1.27 1.27)
+				)
+			)
+		)
 		(pin "J17"
 		)
@@
 			)
 		)
+		(property "LCSC" "C47339"
+			(at 123.19 62.23 0)
+			(effects
+				(font
+					(size 1.27 1.27)
+				)
+			)
+		)
 		(pin "2"
 		)
@@
 			)
 		)
-		(property "Footprint" "Capacitor_SMD:C_1210_3225Metric"
+		(property "Footprint" "Capacitor_SMD:C_1206_3216Metric"
 			(at 331.1652 66.04 0)
 			(effects
@@
 				)
 				(hide yes)
+			)
+		)
+		(property "LCSC" "C96123"
+			(at 330.2 62.23 0)
+			(effects
+				(font
+					(size 1.27 1.27)
+				)
 			)
 		)
@@
 			)
 		)
+		(property "LCSC" "C47339"
+			(at 279.4 62.23 0)
+			(effects
+				(font
+					(size 1.27 1.27)
+				)
+			)
+		)
