File: fpga-pg4.kicad_sch (KiCad schematic)
At the start: 3 parts, among them U1 XC7A35T-FGG484

Commit message: did alot of stuff
Parts:
- C43: footprint Capacitor_SMD:C_1210_3225Metric -> Capacitor_SMD:C_1206_3216Metric; LCSC (none) -> C96123
- R6: footprint Resistor_SMD:R_0402_1005Metric_Pad0.72x0.64mm_HandSolder -> Resistor_SMD:R_0402_1005Metric; LCSC C226391 -> C17168
- U1: LCSC (none) -> C1521727
Changed lines of the file:
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@@
+			)
+		)
+		(property "LCSC" "C1521727"
+			(at 209.55 91.44 0)
+			(effects
+				(font
+					(size 1.27 1.27)
+				)
 			)
 		)
@@
 			)
 		)
-		(property "Footprint" "Capacitor_SMD:C_1210_3225Metric"
+		(property "Footprint" "Capacitor_SMD:C_1206_3216Metric"
 			(at 225.7552 44.45 0)
 			(effects
@@
 				)
 				(hide yes)
+			)
+		)
+		(property "LCSC" "C96123"
+			(at 224.79 40.64 0)
+			(effects
+				(font
+					(size 1.27 1.27)
+				)
 			)
 		)
@@
 			)
 		)
-		(property "Footprint" "Resistor_SMD:R_0402_1005Metric_Pad0.72x0.64mm_HandSolder"
+		(property "Footprint" "Resistor_SMD:R_0402_1005Metric"
 			(at 281.94 85.598 90)
 			(effects
@@
 			)
 		)
-		(property "LCSC" "C226391"
+		(property "LCSC" "C17168"
 			(at 281.94 83.82 0)
 			(effects
@@
 			)
 		)
+		(property "LCSC" "C1521727"
+			(at 209.55 196.85 0)
+			(effects
+				(font
+					(size 1.27 1.27)
+				)
+			)
+		)
