File: frontend_conn.kicad_sch (KiCad schematic)
At the start: 1 part, among them J1 QSH-030-01-X-D-A-XX

Commit message: stuff
Connections:
- net DI.DI2+: now reaches J1.01
- net DI.DI1+: now reaches J1.02
- net DI.DI2-: now reaches J1.03
- net DI.DI1-: now reaches J1.04
- net DI.DI3+: now reaches J1.05
- net DO.DO1+: now reaches J1.06
- net DI.DI3-: now reaches J1.07
- net DO.DO1-: now reaches J1.08
- net DI.DI4+: now reaches J1.09
- net DO.DO2+: now reaches J1.10
- net DI.DI4-: now reaches J1.11
- net DO.DO2-: now reaches J1.12
- net DI.DI5+: now reaches J1.13
- net DO.DO3+: now reaches J1.14
- net DI.DI5-: now reaches J1.15
- net DO.DO3-: now reaches J1.16
- net DI.DI6+: now reaches J1.17
- net DO.DO4+: now reaches J1.18
- net DI.DI6-: now reaches J1.19
- net DO.DO4-: now reaches J1.20
- net DI.DI7+: now reaches J1.21
- net DO.DO5+: now reaches J1.22
- net DI.DI7-: now reaches J1.23
- net DO.DO5-: now reaches J1.24
- net DI.DI8+: now reaches J1.25
- net DO.DO6+: now reaches J1.26
- net DI.DI8-: now reaches J1.27
- net DO.DO6-: now reaches J1.28
- net DI.DI9+: now reaches J1.29
- net DO.DO7+: now reaches J1.30
- net DI.DI9-: now reaches J1.31
- net DO.DO7-: now reaches J1.32
- net DI.DI10+: now reaches J1.33
- net DO.DO8+: now reaches J1.34
- net DI.DI10-: now reaches J1.35
- net DO.DO8-: now reaches J1.36
- net DI.DI11+: now reaches J1.37
- net DI.DI11-: now reaches J1.39
- net DI.DI12+: now reaches J1.41
- net DI.DI12-: now reaches J1.43
- net DI.DI13+: now reaches J1.45
- net DI.DI13-: now reaches J1.47
- net DI.DI14+: now reaches J1.49
- net DI.DI14-: now reaches J1.51
- net DI.DI15+: now reaches J1.53
- net DI.DI15-: now reaches J1.55
- net DI.DI16+: now reaches J1.57
- net DI.DI16-: now reaches J1.59

Commit message: added a lot of stuff
Connections:
- net I2C.DATA: now reaches J1.38
- net I2C.CLK: now reaches J1.40
- net INT#: now reaches J1.42
- net VBUS: now reaches J1.44
- net VBUS: now also J1.46
- net +3.3V: now reaches J1.48
- net +3.3V: now also J1.50
- net +1V8: now reaches J1.52
- net +1V5: now reaches J1.54
- net GND: now reaches J1.56
- net GND: now also J1.58, J1.60, J1.G1, J1.G2, J1.G3, J1.G4

Commit message: started doing some general floorplanning and outline
Parts:
- added H1, H2, H3, H4: MountingHole_Pad, MountingHole:MountingHole_3.2mm_M3, symbol Mechanical:MountingHole_Pad
Connections:
- net GND: now also H1.1, H2.1, H3.1, H4.1

Commit message: more floorplanning
Parts:
- H1, H2, H3, H4: footprint MountingHole:MountingHole_3.2mm_M3 -> MountingHole:MountingHole_3.2mm_M3_DIN965_Pad
Changed lines of the file:
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@@
 			)
 		)
-		(property "Footprint" "MountingHole:MountingHole_3.2mm_M3"
+		(property "Footprint" "MountingHole:MountingHole_3.2mm_M3_DIN965_Pad"
 			(at 68.58 130.81 0)
 			(effects
@@
 			)
 		)
-		(property "Footprint" "MountingHole:MountingHole_3.2mm_M3"
+		(property "Footprint" "MountingHole:MountingHole_3.2mm_M3_DIN965_Pad"
 			(at 68.58 116.84 0)
 			(effects
@@
 			)
 		)
-		(property "Footprint" "MountingHole:MountingHole_3.2mm_M3"
+		(property "Footprint" "MountingHole:MountingHole_3.2mm_M3_DIN965_Pad"
 			(at 68.58 102.87 0)
 			(effects
@@
 			)
 		)
-		(property "Footprint" "MountingHole:MountingHole_3.2mm_M3"
+		(property "Footprint" "MountingHole:MountingHole_3.2mm_M3_DIN965_Pad"
 			(at 68.58 88.9 0)
 			(effects

Commit message: did alot of stuff
Parts:
- J1: LCSC (none) -> C5714556
Changed lines of the file:
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@@
+			)
+		)
+		(property "LCSC" "C5714556"
+			(at 153.67 95.25 0)
+			(effects
+				(font
+					(size 1.27 1.27)
+				)
 			)
 		)
