File: pmic.kicad_sch (KiCad schematic)
At the start: 1 part, among them U2 MP5470GL-0000-P

Commit message: more stuff!
Parts:
- added C16, C17, C19, C20, C21, C22: 22u, Capacitor_SMD:C_0603_1608Metric, symbol Device:C
- added C18: 1u, Capacitor_SMD:C_0402_1005Metric, symbol Device:C
- added L1, L2, L3, L4: 2.2u, Inductor_SMD:L_Bourns-SRN4018, symbol Device:L
- added R1: 10k, Resistor_SMD:R_0402_1005Metric, symbol Device:R
- U2: footprint QFN-3x4_MP5470_MNP -> MP5470:QFN-3x4_MP5470_MNP
Connections:
- net VIN: now reaches U2.1 (VIN1)
- net VIN: now also U2.5 (VIN2), C16.1, C17.1
- net at U2.10 (FB3): now also C21.1, L3.2
- net at U2.13 (SW3): now also L3.1
- net at U2.15 (SW4): now also L4.1
- net at U2.16 (VCC): now also C18.1, R1.1
- net at U2.18 (FB4): now also C22.1, L4.2
- net at U2.2 (SW1): now also L1.1
- net at U2.20 (GPIO): now also R1.2
- net GND: now reaches U2.21 (SGND1)
- net GND: now also U2.9 (SGND2), C16.2, C17.2, C18.2, C19.2, C20.2, C21.2, C22.2
- net at U2.22 (FB1): now also C19.1, L1.2
- net at U2.4 (SW2): now also L2.1
- net at U2.6 (FB2): now also C20.1, L2.2
Other:
- moved on the sheet: U2

Commit message: stuff
Parts:
- added TP33, TP34, TP35, TP36, TP37, TP38, TP39, TP40, TP41: TestPoint, symbol Connector:TestPoint
- added TP42: TestPoint_Alt, symbol Connector:TestPoint_Alt
Connections:
- net GND: now also U2.14 (GND), U2.19 (AGND), U2.3 (GND), TP42.1
- net +1V5: now reaches C22.1, L4.2, U2.18 (FB4)
- net +1V5: now also TP36.1
- net +3.3V: now reaches C20.1, L2.2, U2.6 (FB2)
- net +3.3V: now also TP34.1
- net VCCINT: now reaches C19.1, L1.2, U2.22 (FB1)
- net VCCINT: now also TP33.1
- net at C18.1, R1.1, U2.16 (VCC): now also TP38.1
- net +1V8: now reaches C21.1, L3.2, U2.10 (FB3)
- net +1V8: now also TP35.1
- net EN: now reaches U2.12 (EN/SYNC)
- net EN: now also TP41.1
- net I2C.SCL: now reaches U2.7 (SCL)
- net I2C.SCL: now also TP39.1
- net I2C.SDA: now reaches U2.8 (SDA)
- net I2C.SDA: now also TP40.1
- net VIN renamed VBUS
- net VBUS: now also TP37.1
Other:
- note added: "ARTIX 7 PMIC"
- moved on the sheet: C16, C17, C18, C19, C20, C21, C22, L1, L2, L3, L4, R1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

Commit message: added a lot of stuff
Parts:
- renumbered C19 to C44, C17 to C45, C16 to C46, C18 to C47, C20 to C48, C21 to C49, C22 to C50, R1 to R7, TP37 to TP49, TP33 to TP50, TP38 to TP51, TP34 to TP52, TP39 to TP53, TP40 to TP54, TP35 to TP55, TP41 to TP56, TP36 to TP57, TP42 to TP58
Other:
- note added: "TODO: check overall current draw"

Commit message: did alot of stuff
Parts:
- C44, C45, C46, C48, C49, C50: LCSC (none) -> C59461
- C47: LCSC (none) -> C52923
- L1, L2, L3, L4: LCSC (none) -> C913207
- R7: LCSC (none) -> C25744
- TP49, TP50, TP51, TP52, TP53, TP54, TP55, TP56, TP57, TP58: now not fitted
Changed lines of the file:
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@@
+			)
+		)
+		(property "LCSC" "C59461"
+			(at 200.66 132.08 0)
+			(effects
+				(font
+					(size 1.27 1.27)
+				)
 			)
 		)
@@
 		(in_bom yes)
 		(on_board yes)
-		(dnp no)
+		(dnp yes)
 		(fields_autoplaced yes)
 		(property "Reference" "TP55"
@@
 		(in_bom yes)
 		(on_board yes)
-		(dnp no)
+		(dnp yes)
 		(property "Reference" "TP54"
 			(at 120.142 96.774 90)
@@
 		(in_bom yes)
 		(on_board yes)
-		(dnp no)
+		(dnp yes)
 		(fields_autoplaced yes)
 		(property "Reference" "TP52"
@@
 		(in_bom yes)
 		(on_board yes)
-		(dnp no)
+		(dnp yes)
 		(property "Reference" "TP56"
 			(at 120.142 105.664 90)
@@
 		(in_bom yes)
 		(on_board yes)
-		(dnp no)
+		(dnp yes)
 		(property "Reference" "TP53"
 			(at 120.142 94.234 90)
@@
 			)
 		)
+		(property "LCSC" "C913207"
+			(at 189.23 127 0)
+			(effects
+				(font
+					(size 1.27 1.27)
+				)
+			)
+		)
 		(pin "1"
 		)
@@
 			)
 		)
+		(property "LCSC" "C59461"
+			(at 200.66 88.9 0)
+			(effects
+				(font
+					(size 1.27 1.27)
+				)
+			)
+		)
 		(pin "2"
 		)
@@
 		(in_bom yes)
 		(on_board yes)
-		(dnp no)
+		(dnp yes)
 		(fields_autoplaced yes)
 		(property "Reference" "TP58"
@@
 			)
 		)
+		(property "LCSC" "C59461"
+			(at 200.66 67.31 0)
+			(effects
+				(font
+					(size 1.27 1.27)
+				)
+			)
+		)
 		(pin "2"
 		)
@@
 			)
 		)
+		(property "LCSC" "C59461"
+			(at 87.63 68.58 0)
+			(effects
+				(font
+					(size 1.27 1.27)
+				)
+			)
+		)
 		(pin "2"
 		)
@@
 			)
 		)
+		(property "LCSC" "C25744"
+			(at 123.19 81.28 0)
+			(effects
+				(font
+					(size 1.27 1.27)
+				)
+			)
+		)
 		(pin "1"
 		)
@@
 			)
 		)
+		(property "LCSC" "C913207"
+			(at 189.23 83.82 0)
+			(effects
+				(font
+					(size 1.27 1.27)
+				)
+			)
+		)
 		(pin "1"
 		)
@@
 			)
 		)
+		(property "LCSC" "C913207"
+			(at 189.23 105.41 0)
+			(effects
+				(font
+					(size 1.27 1.27)
+				)
+			)
+		)
 		(pin "1"
 		)
@@
 			)
 		)
+		(property "LCSC" "C59461"
+			(at 99.06 68.58 0)
+			(effects
+				(font
+					(size 1.27 1.27)
+				)
+			)
+		)
 		(pin "2"
 		)
@@
 		(in_bom yes)
 		(on_board yes)
-		(dnp no)
+		(dnp yes)
 		(fields_autoplaced yes)
 		(property "Reference" "TP51"
@@
 			)
 		)
+		(property "LCSC" "C913207"
+			(at 189.23 62.23 0)
+			(effects
+				(font
+					(size 1.27 1.27)
+				)
+			)
+		)
 		(pin "1"
 		)
@@
 		(in_bom yes)
 		(on_board yes)
-		(dnp no)
+		(dnp yes)
 		(fields_autoplaced yes)
 		(property "Reference" "TP57"
@@
 			)
 		)
+		(property "LCSC" "C52923"
+			(at 110.49 81.28 0)
+			(effects
+				(font
+					(size 1.27 1.27)
+				)
+			)
+		)
 		(pin "2"
 		)
@@
 		(in_bom yes)
 		(on_board yes)
-		(dnp no)
+		(dnp yes)
 		(fields_autoplaced yes)
 		(property "Reference" "TP49"
@@
 		(in_bom yes)
 		(on_board yes)
-		(dnp no)
+		(dnp yes)
 		(fields_autoplaced yes)
 		(property "Reference" "TP50"
@@
 			)
 		)
+		(property "LCSC" "C59461"
+			(at 200.66 110.49 0)
+			(effects
+				(font
+					(size 1.27 1.27)
+				)
+			)
+		)
