File: spi_flash.kicad_sch (KiCad schematic)
At the start: 0 parts

Commit message: more stuff
Parts:
- added C29: 100n, symbol Device:C
- added TP10, TP11, TP12, TP13, TP14, TP16: TestPoint, symbol Connector:TestPoint
- added TP15: TestPoint_Alt, symbol Connector:TestPoint_Alt
- added U5: MX25L3233FZN, Package_SON:WSON-8-1EP_6x5mm_P1.27mm_EP3.4x4mm, symbol Memory_Flash:MX25L3233FZN
Connections:
- new net: C29.1, U5.8 (VCC)
- new net FLASH_SPI.CLK: TP16.1, U5.6 (SCLK)
- new net FLASH_SPI.CS#: TP10.1, U5.1 (~{CS})
- new net FLASH_SPI.D0: TP11.1, U5.5 (SI/SIO0)
- new net FLASH_SPI.D1: TP12.1, U5.2 (SO/SIO1)
- new net FLASH_SPI.D2: TP13.1, U5.3 (~{WP}/SIO2)
- new net FLASH_SPI.D3: TP14.1, U5.7 (~{HOLD}/SIO3)
- new net GND: C29.2, TP15.1, U5.4 (GND), U5.9 (EP)
Other:
- note added: "PROGRAM FLASH"
- note added: "TODO: connect vcc"

Commit message: working on ddr3
Parts:
- C29: footprint (none) -> Capacitor_SMD:C_0402_1005Metric
Changed lines of the file:
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@@
 			)
 		)
-		(property "Footprint" ""
+		(property "Footprint" "Capacitor_SMD:C_0402_1005Metric"
 			(at 173.6852 85.09 0)
 			(effects

Commit message: added a lot of stuff
Parts:
- renumbered C29 to C57, TP10 to TP68, TP16 to TP69, TP11 to TP70, TP12 to TP71, TP13 to TP72, TP14 to TP73, TP15 to TP74
Changed lines of the file:
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@@
 		(dnp no)
 		(fields_autoplaced yes)
-		(property "Reference" "C29"
+		(property "Reference" "C57"
 			(at 176.53 80.0099 0)
 			(effects
@@
 			(project "logix-core"
 				(path "/cf3b7c5f-6ddc-4e3f-9529-0bcf5eec6f23/b85739df-cd60-41d1-92dc-c1028520afa1"
-					(reference "C29")
+					(reference "C57")
 					(unit 1)
 				)
@@
 		(dnp no)
 		(fields_autoplaced yes)
-		(property "Reference" "#PWR039"
+		(property "Reference" "#PWR046"
 			(at 156.21 114.3 0)
 			(effects
@@
 			(project "logix-core"
 				(path "/cf3b7c5f-6ddc-4e3f-9529-0bcf5eec6f23/b85739df-cd60-41d1-92dc-c1028520afa1"
-					(reference "#PWR039")
+					(reference "#PWR046")
 					(unit 1)
 				)
@@
 		(on_board yes)
 		(dnp no)
-		(property "Reference" "TP12"
+		(property "Reference" "TP71"
 			(at 137.668 91.694 90)
 			(effects
@@
 			(project "logix-core"
 				(path "/cf3b7c5f-6ddc-4e3f-9529-0bcf5eec6f23/b85739df-cd60-41d1-92dc-c1028520afa1"
-					(reference "TP12")
+					(reference "TP71")
 					(unit 1)
 				)
@@
 		(on_board yes)
 		(dnp no)
-		(property "Reference" "TP13"
+		(property "Reference" "TP72"
 			(at 137.668 94.234 90)
 			(effects
@@
 			(project "logix-core"
 				(path "/cf3b7c5f-6ddc-4e3f-9529-0bcf5eec6f23/b85739df-cd60-41d1-92dc-c1028520afa1"
-					(reference "TP13")
+					(reference "TP72")
 					(unit 1)
 				)
@@
 		(dnp no)
 		(fields_autoplaced yes)
-		(property "Reference" "#PWR038"
+		(property "Reference" "#PWR047"
 			(at 172.72 118.11 0)
 			(effects
@@
 			(project "logix-core"
 				(path "/cf3b7c5f-6ddc-4e3f-9529-0bcf5eec6f23/b85739df-cd60-41d1-92dc-c1028520afa1"
-					(reference "#PWR038")
+					(reference "#PWR047")
 					(unit 1)
 				)
@@
 		(dnp no)
 		(fields_autoplaced yes)
-		(property "Reference" "#PWR037"
+		(property "Reference" "#PWR045"
 			(at 172.72 92.71 0)
 			(effects
@@
 			(project "logix-core"
 				(path "/cf3b7c5f-6ddc-4e3f-9529-0bcf5eec6f23/b85739df-cd60-41d1-92dc-c1028520afa1"
-					(reference "#PWR037")
+					(reference "#PWR045")
 					(unit 1)
 				)
@@
 		(on_board yes)
 		(dnp no)
-		(property "Reference" "TP11"
+		(property "Reference" "TP70"
 			(at 137.668 89.154 90)
 			(effects
@@
 			(project "logix-core"
 				(path "/cf3b7c5f-6ddc-4e3f-9529-0bcf5eec6f23/b85739df-cd60-41d1-92dc-c1028520afa1"
-					(reference "TP11")
+					(reference "TP70")
 					(unit 1)
 				)
@@
 		(on_board yes)
 		(dnp no)
-		(property "Reference" "TP10"
+		(property "Reference" "TP68"
 			(at 137.668 84.074 90)
 			(effects
@@
 			(project "logix-core"
 				(path "/cf3b7c5f-6ddc-4e3f-9529-0bcf5eec6f23/b85739df-cd60-41d1-92dc-c1028520afa1"
-					(reference "TP10")
+					(reference "TP68")
 					(unit 1)
 				)
@@
 		(on_board yes)
 		(dnp no)
-		(property "Reference" "TP16"
+		(property "Reference" "TP69"
 			(at 137.668 86.614 90)
 			(effects
@@
 			(project "logix-core"
 				(path "/cf3b7c5f-6ddc-4e3f-9529-0bcf5eec6f23/b85739df-cd60-41d1-92dc-c1028520afa1"
-					(reference "TP16")
+					(reference "TP69")
 					(unit 1)
 				)
@@
 		(on_board yes)
 		(dnp no)
-		(property "Reference" "TP14"
+		(property "Reference" "TP73"
 			(at 137.668 96.774 90)
 			(effects
@@
 			(project "logix-core"
 				(path "/cf3b7c5f-6ddc-4e3f-9529-0bcf5eec6f23/b85739df-cd60-41d1-92dc-c1028520afa1"
-					(reference "TP14")
+					(reference "TP73")
 					(unit 1)
 				)
@@
 		(dnp no)
 		(fields_autoplaced yes)
-		(property "Reference" "TP15"
+		(property "Reference" "TP74"
 			(at 175.26 107.1879 0)
 			(effects
@@
 			(project "logix-core"
 				(path "/cf3b7c5f-6ddc-4e3f-9529-0bcf5eec6f23/b85739df-cd60-41d1-92dc-c1028520afa1"
-					(reference "TP15")
-					(unit 1)
-				)
+					(reference "TP74")
+					(unit 1)
+				)

Commit message: did alot of stuff
Parts:
- C57: LCSC (none) -> C1525
- TP68, TP69, TP70, TP71, TP72, TP73, TP74: now not fitted
Changed lines of the file:
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@@
+			)
+		)
+		(property "LCSC" "C1525"
+			(at 172.72 81.28 0)
+			(effects
+				(font
+					(size 1.27 1.27)
+				)
 			)
 		)
@@
 		(in_bom yes)
 		(on_board yes)
-		(dnp no)
+		(dnp yes)
 		(property "Reference" "TP71"
 			(at 137.668 91.694 90)
@@
 		(in_bom yes)
 		(on_board yes)
-		(dnp no)
+		(dnp yes)
 		(property "Reference" "TP72"
 			(at 137.668 94.234 90)
@@
 		(in_bom yes)
 		(on_board yes)
-		(dnp no)
+		(dnp yes)
 		(property "Reference" "TP70"
 			(at 137.668 89.154 90)
@@
 		(in_bom yes)
 		(on_board yes)
-		(dnp no)
+		(dnp yes)
 		(property "Reference" "TP68"
 			(at 137.668 84.074 90)
@@
 		(in_bom yes)
 		(on_board yes)
-		(dnp no)
+		(dnp yes)
 		(property "Reference" "TP69"
 			(at 137.668 86.614 90)
@@
 		(in_bom yes)
 		(on_board yes)
-		(dnp no)
+		(dnp yes)
 		(property "Reference" "TP73"
 			(at 137.668 96.774 90)
@@
 		(in_bom yes)
 		(on_board yes)
-		(dnp no)
+		(dnp yes)
 		(fields_autoplaced yes)
 		(property "Reference" "TP74"
