File: usb.kicad_sch (KiCad schematic)
At the start: 30 parts, among them U3 TPUSBLC6-4SC6, U4 FT230XQ

Commit message: added a lot of stuff
Parts:
- renumbered C27 to C51, C28 to C52, C26 to C53, C25 to C54, C24 to C55, C23 to C56, R6 to R10, R2 to R11, R7 to R12, R3 to R13, R10 to R14, R8 to R15, R9 to R16, R4 to R8, R5 to R9, TP8 to TP59, TP6 to TP60, TP7 to TP61, TP2 to TP62, TP9 to TP63, TP3 to TP64, TP4 to TP65, TP1 to TP66, TP5 to TP67

Commit message: more floorplanning
Parts:
- D1, D2: footprint LED_SMD:LED_0603_1608Metric -> LED_SMD:LED_0805_2012Metric
Changed lines of the file:
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@@
 			)
 		)
-		(property "Footprint" "LED_SMD:LED_0603_1608Metric"
+		(property "Footprint" "LED_SMD:LED_0805_2012Metric"
 			(at 257.81 133.35 0)
 			(effects
@@
 			)
 		)
-		(property "Footprint" "LED_SMD:LED_0603_1608Metric"
+		(property "Footprint" "LED_SMD:LED_0805_2012Metric"
 			(at 241.3 133.35 0)
 			(effects

Commit message: did alot of stuff
Parts:
- C51, C52, C53: LCSC (none) -> C1525
- C54: LCSC (none) -> C15195
- C55, C56: LCSC (none) -> C1567
- D1, D2: LCSC (none) -> C2297
- R10, R12, R8, R9: footprint Resistor_SMD:R_0402_1005Metric_Pad0.72x0.64mm_HandSolder -> Resistor_SMD:R_0402_1005Metric; LCSC C226391 -> C17168
- R11, R13: footprint Resistor_SMD:R_0402_1005Metric_Pad0.72x0.64mm_HandSolder -> Resistor_SMD:R_0402_1005Metric
- R14, R15, R16: footprint Resistor_SMD:R_0402_1005Metric_Pad0.72x0.64mm_HandSolder -> Resistor_SMD:R_0402_1005Metric; LCSC C226391 -> C25076
- TP59, TP60, TP61, TP62, TP63, TP64, TP65, TP66, TP67: now not fitted
- U4: LCSC (none) -> C128629
- USB1: LCSC (none) -> C2927008
Connections:
- net EXT_VBUS: now reaches C54.1, FB1.1, USB1.1 (VCC)
Other:
- note added: "TODO: add jumper for VBUS power"
Changed lines of the file:
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@@
 		)
 	)
+	(text "TODO: add jumper for VBUS power"
+		(exclude_from_sim no)
+		(at 177.038 55.372 0)
+		(effects
+			(font
+				(size 1.27 1.27)
+			)
+		)
+	)
 	(text "TODO: connect reset"
 		(exclude_from_sim no)
@@
 		)
 	)
+	(label "EXT_VBUS"
+		(at 62.23 59.69 0)
+		(effects
+			(font
+				(size 1.27 1.27)
+			)
+			(justify left bottom)
+		)
+	)
 	(label "FTDI_TXD"
 		(at 190.5 93.98 0)
@@
 			)
 		)
-		(property "Footprint" "Resistor_SMD:R_0402_1005Metric_Pad0.72x0.64mm_HandSolder"
+		(property "Footprint" "Resistor_SMD:R_0402_1005Metric"
 			(at 209.55 98.298 90)
 			(effects
@@
 			)
 		)
-		(property "LCSC" "C226391"
+		(property "LCSC" "C17168"
 			(at 209.55 96.52 0)
 			(effects
@@
 			)
 		)
+		(property "LCSC" "C1525"
+			(at 140.97 86.36 0)
+			(effects
+				(font
+					(size 1.27 1.27)
+				)
+			)
+		)
 		(pin "2"
 		)
@@
 		(in_bom yes)
 		(on_board yes)
-		(dnp no)
+		(dnp yes)
 		(fields_autoplaced yes)
 		(property "Reference" "TP63"
@@
 			)
 		)
-		(property "Footprint" "Resistor_SMD:R_0402_1005Metric_Pad0.72x0.64mm_HandSolder"
+		(property "Footprint" "Resistor_SMD:R_0402_1005Metric"
 			(at 150.368 118.11 90)
 			(effects
@@
 			)
 		)
-		(property "LCSC" "C226391"
+		(property "LCSC" "C25076"
 			(at 148.59 118.11 0)
 			(effects
@@
 			)
 		)
+		(property "LCSC" "C15195"
+			(at 60.96 115.57 0)
+			(effects
+				(font
+					(size 1.27 1.27)
+				)
+			)
+		)
 		(pin "2"
 		)
@@
 			)
 		)
-		(property "Footprint" "Resistor_SMD:R_0402_1005Metric_Pad0.72x0.64mm_HandSolder"
+		(property "Footprint" "Resistor_SMD:R_0402_1005Metric"
 			(at 243.078 121.92 90)
 			(effects
@@
 			)
 		)
-		(property "LCSC" "C226391"
+		(property "LCSC" "C25076"
 			(at 241.3 121.92 0)
 			(effects
@@
 		(in_bom yes)
 		(on_board yes)
-		(dnp no)
+		(dnp yes)
 		(fields_autoplaced yes)
 		(property "Reference" "TP64"
@@
 			)
 		)
+		(property "LCSC" "C2297"
+			(at 257.81 133.35 0)
+			(effects
+				(font
+					(size 1.27 1.27)
+				)
+			)
+		)
 		(pin "2"
 		)
@@
 		(in_bom yes)
 		(on_board yes)
-		(dnp no)
+		(dnp yes)
 		(fields_autoplaced yes)
 		(property "Reference" "TP61"
@@
 			)
 		)
+		(property "LCSC" "C1525"
+			(at 157.48 74.93 0)
+			(effects
+				(font
+					(size 1.27 1.27)
+				)
+			)
+		)
 		(pin "2"
 		)
@@
 			)
 		)
+		(property "LCSC" "C2927008"
+			(at 46.99 104.14 0)
+			(effects
+				(font
+					(size 1.27 1.27)
+				)
+			)
+		)
 		(pin "5"
 		)
@@
 			)
 		)
-		(property "Footprint" "Resistor_SMD:R_0402_1005Metric_Pad0.72x0.64mm_HandSolder"
+		(property "Footprint" "Resistor_SMD:R_0402_1005Metric"
 			(at 209.55 103.378 90)
 			(effects
@@
 			)
 		)
-		(property "LCSC" "C226391"
+		(property "LCSC" "C17168"
 			(at 209.55 101.6 0)
 			(effects
@@
 			)
 		)
-		(property "Footprint" "Resistor_SMD:R_0402_1005Metric_Pad0.72x0.64mm_HandSolder"
+		(property "Footprint" "Resistor_SMD:R_0402_1005Metric"
 			(at 125.73 105.918 90)
 			(effects
@@
 			)
 		)
+		(property "LCSC" "C2297"
+			(at 241.3 133.35 0)
+			(effects
+				(font
+					(size 1.27 1.27)
+				)
+			)
+		)
 		(pin "2"
 		)
@@
 			)
 		)
+		(property "LCSC" "C1567"
+			(at 99.06 115.57 0)
+			(effects
+				(font
+					(size 1.27 1.27)
+				)
+			)
+		)
 		(pin "2"
 		)
@@
 			)
 		)
-		(property "Footprint" "Resistor_SMD:R_0402_1005Metric_Pad0.72x0.64mm_HandSolder"
+		(property "Footprint" "Resistor_SMD:R_0402_1005Metric"
 			(at 259.588 121.92 90)
 			(effects
@@
 			)
 		)
-		(property "LCSC" "C226391"
+		(property "LCSC" "C25076"
 			(at 257.81 121.92 0)
 			(effects
@@
 		(in_bom yes)
 		(on_board yes)
-		(dnp no)
+		(dnp yes)
 		(property "Reference" "TP59"
 			(at 119.38 57.6579 0)
@@
 		(in_bom yes)
 		(on_board yes)
-		(dnp no)
+		(dnp yes)
 		(fields_autoplaced yes)
 		(property "Reference" "TP65"
@@
 			)
 		)
+		(property "LCSC" "C1567"
+			(at 111.76 115.57 0)
+			(effects
+				(font
+					(size 1.27 1.27)
+				)
+			)
+		)
 		(pin "1"
 		)
@@
 		(in_bom yes)
 		(on_board yes)
-		(dnp no)
+		(dnp yes)
 		(property "Reference" "TP60"
 			(at 88.9 95.7579 0)
@@
 		(in_bom yes)
 		(on_board yes)
-		(dnp no)
+		(dnp yes)
 		(fields_autoplaced yes)
 		(property "Reference" "TP66"
@@
 			)
 		)
-		(property "Footprint" "Resistor_SMD:R_0402_1005Metric_Pad0.72x0.64mm_HandSolder"
+		(property "Footprint" "Resistor_SMD:R_0402_1005Metric"
 			(at 209.55 95.758 90)
 			(effects
@@
 			)
 		)
-		(property "LCSC" "C226391"
+		(property "LCSC" "C17168"
 			(at 209.55 93.98 0)
 			(effects
@@
 			)
 		)
+		(property "LCSC" "C1525"
+			(at 187.96 74.93 0)
+			(effects
+				(font
+					(size 1.27 1.27)
+				)
+			)
+		)
 		(pin "2"
 		)
@@
 			)
 		)
+		(property "LCSC" "C128629"
+			(at 170.18 104.14 0)
+			(effects
+				(font
+					(size 1.27 1.27)
+				)
+			)
+		)
 		(pin "8"
 		)
@@
 			)
 		)
-		(property "Footprint" "Resistor_SMD:R_0402_1005Metric_Pad0.72x0.64mm_HandSolder"
+		(property "Footprint" "Resistor_SMD:R_0402_1005Metric"
 			(at 209.55 100.838 90)
 			(effects
@@
 			)
 		)
-		(property "LCSC" "C226391"
+		(property "LCSC" "C17168"
 			(at 209.55 99.06 0)
 			(effects
@@
 			)
 		)
-		(property "Footprint" "Resistor_SMD:R_0402_1005Metric_Pad0.72x0.64mm_HandSolder"
+		(property "Footprint" "Resistor_SMD:R_0402_1005Metric"
 			(at 125.73 103.378 90)
 			(effects
@@
 		(in_bom yes)
 		(on_board yes)
-		(dnp no)
+		(dnp yes)
 		(fields_autoplaced yes)
 		(property "Reference" "TP67"
@@
 		(in_bom yes)
 		(on_board yes)
-		(dnp no)
+		(dnp yes)
 		(fields_autoplaced yes)
 		(property "Reference" "TP62"
