File: ddr3.kicad_sch (KiCad schematic)
At the start: 11 parts, among them U8 MT41K256M16TW-107:P

Commit message: added a lot of stuff
Parts:
- renumbered C42 to C58, C41 to C59, C40 to C60, C36 to C61, C39 to C62, C37 to C63, C38 to C64, R19 to R17, R20 to R18, R18 to R19, U8 to U6
Changed lines of the file:
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@@
+		(polyline
+			(pts
+				(xy 137.16 69.85) (xy 137.16 88.9) (xy 144.78 88.9) (xy 144.78 69.85)
+			)
+			(stroke
+				(width 0)
+				(type dash)
+			)
+			(fill
+				(type none)
+			)
+		)
+	)
+	(rule_area
+		(polyline
+			(pts
+				(xy 137.16 45.72) (xy 137.16 67.31) (xy 144.78 67.31) (xy 144.78 45.72)
+			)
+			(stroke
+				(width 0)
+				(type dash)
+			)
+			(fill
+				(type none)
+			)
+		)
+	)
+	(rule_area
 		(polyline
 			(pts
@@
 			(pts
 				(xy 82.55 116.84) (xy 82.55 129.54) (xy 87.63 129.54) (xy 87.63 116.84)
-			)
-			(stroke
-				(width 0)
-				(type dash)
-			)
-			(fill
-				(type none)
-			)
-		)
-	)
-	(rule_area
-		(polyline
-			(pts
-				(xy 137.16 45.72) (xy 137.16 67.31) (xy 144.78 67.31) (xy 144.78 45.72)
-			)
-			(stroke
-				(width 0)
-				(type dash)
-			)
-			(fill
-				(type none)
-			)
-		)
-	)
-	(rule_area
-		(polyline
-			(pts
-				(xy 137.16 69.85) (xy 137.16 88.9) (xy 144.78 88.9) (xy 144.78 69.85)
 			)
 			(stroke
@@
 		(on_board yes)
 		(dnp no)
-		(property "Reference" "R18"
+		(property "Reference" "R19"
 			(at 76.2 152.3999 0)
 			(effects
@@
 			(project "logix-core"
 				(path "/cf3b7c5f-6ddc-4e3f-9529-0bcf5eec6f23/ab2b6d75-2b5d-47d9-b70e-fad58fb7011e"
-					(reference "R18")
+					(reference "R19")
 					(unit 1)
 				)
@@
 		(dnp no)
 		(fields_autoplaced yes)
-		(property "Reference" "#PWR058"
+		(property "Reference" "#PWR054"
 			(at 175.26 110.49 0)
 			(effects
@@
 			(project "logix-core"
 				(path "/cf3b7c5f-6ddc-4e3f-9529-0bcf5eec6f23/ab2b6d75-2b5d-47d9-b70e-fad58fb7011e"
-					(reference "#PWR058")
+					(reference "#PWR054")
 					(unit 1)
 				)
@@
 		(dnp no)
 		(fields_autoplaced yes)
-		(property "Reference" "#PWR055"
+		(property "Reference" "#PWR052"
 			(at 208.28 63.5 0)
 			(effects
@@
 			(project "logix-core"
 				(path "/cf3b7c5f-6ddc-4e3f-9529-0bcf5eec6f23/ab2b6d75-2b5d-47d9-b70e-fad58fb7011e"
-					(reference "#PWR055")
+					(reference "#PWR052")
 					(unit 1)
 				)
@@
 		(dnp no)
 		(fields_autoplaced yes)
-		(property "Reference" "#PWR057"
+		(property "Reference" "#PWR055"
 			(at 186.69 110.49 0)
 			(effects
@@
 			(project "logix-core"
 				(path "/cf3b7c5f-6ddc-4e3f-9529-0bcf5eec6f23/ab2b6d75-2b5d-47d9-b70e-fad58fb7011e"
-					(reference "#PWR057")
+					(reference "#PWR055")
 					(unit 1)
 				)
@@
 		(dnp no)
 		(fields_autoplaced yes)
-		(property "Reference" "C40"
+		(property "Reference" "C60"
 			(at 201.93 50.7999 0)
 			(effects
@@
 			(project "logix-core"
 				(path "/cf3b7c5f-6ddc-4e3f-9529-0bcf5eec6f23/ab2b6d75-2b5d-47d9-b70e-fad58fb7011e"
-					(reference "C40")
+					(reference "C60")
 					(unit 1)
 				)
@@
 		(dnp no)
 		(fields_autoplaced yes)
-		(property "Reference" "#PWR062"
+		(property "Reference" "#PWR049"
 			(at 177.8 63.5 0)
 			(effects
@@
 			(project "logix-core"
 				(path "/cf3b7c5f-6ddc-4e3f-9529-0bcf5eec6f23/ab2b6d75-2b5d-47d9-b70e-fad58fb7011e"
-					(reference "#PWR062")
+					(reference "#PWR049")
 					(unit 1)
 				)
@@
 		(dnp no)
 		(fields_autoplaced yes)
-		(property "Reference" "U8"
+		(property "Reference" "U6"
 			(at 111.76 36.83 0)
 			(effects
@@
 			(project "logix-core"
 				(path "/cf3b7c5f-6ddc-4e3f-9529-0bcf5eec6f23/ab2b6d75-2b5d-47d9-b70e-fad58fb7011e"
-					(reference "U8")
+					(reference "U6")
 					(unit 1)
 				)
@@
 		(dnp no)
 		(fields_autoplaced yes)
-		(property "Reference" "#PWR09"
+		(property "Reference" "#PWR059"
 			(at 88.9 165.1 0)
 			(effects
@@
 			(project "logix-core"
 				(path "/cf3b7c5f-6ddc-4e3f-9529-0bcf5eec6f23/ab2b6d75-2b5d-47d9-b70e-fad58fb7011e"
-					(reference "#PWR09")
+					(reference "#PWR059")
 					(unit 1)
 				)
@@
 		(dnp no)
 		(fields_autoplaced yes)
-		(property "Reference" "C38"
+		(property "Reference" "C64"
 			(at 201.93 97.7899 0)
 			(effects
@@
 			(project "logix-core"
 				(path "/cf3b7c5f-6ddc-4e3f-9529-0bcf5eec6f23/ab2b6d75-2b5d-47d9-b70e-fad58fb7011e"
-					(reference "C38")
+					(reference "C64")
 					(unit 1)
 				)
@@
 		(dnp no)
 		(fields_autoplaced yes)
-		(property "Reference" "#PWR061"
+		(property "Reference" "#PWR050"
 			(at 187.96 63.5 0)
 			(effects
@@
 			(project "logix-core"
 				(path "/cf3b7c5f-6ddc-4e3f-9529-0bcf5eec6f23/ab2b6d75-2b5d-47d9-b70e-fad58fb7011e"
-					(reference "#PWR061")
+					(reference "#PWR050")
 					(unit 1)
 				)
@@
 		(dnp no)
 		(fields_autoplaced yes)
-		(property "Reference" "C41"
+		(property "Reference" "C59"
 			(at 191.77 50.7999 0)
 			(effects
@@
 			(project "logix-core"
 				(path "/cf3b7c5f-6ddc-4e3f-9529-0bcf5eec6f23/ab2b6d75-2b5d-47d9-b70e-fad58fb7011e"
-					(reference "C41")
+					(reference "C59")
 					(unit 1)
 				)
@@
 		(dnp no)
 		(fields_autoplaced yes)
-		(property "Reference" "#PWR012"
+		(property "Reference" "#PWR057"
 			(at 224.79 161.29 0)
 			(effects
@@
 			(project "logix-core"
 				(path "/cf3b7c5f-6ddc-4e3f-9529-0bcf5eec6f23/ab2b6d75-2b5d-47d9-b70e-fad58fb7011e"
-					(reference "#PWR012")
+					(reference "#PWR057")
 					(unit 1)
 				)
@@
 		(dnp no)
 		(fields_autoplaced yes)
-		(property "Reference" "#PWR059"
+		(property "Reference" "#PWR053"
 			(at 208.28 83.82 0)
 			(effects
@@
 			(project "logix-core"
 				(path "/cf3b7c5f-6ddc-4e3f-9529-0bcf5eec6f23/ab2b6d75-2b5d-47d9-b70e-fad58fb7011e"
-					(reference "#PWR059")
+					(reference "#PWR053")
 					(unit 1)
 				)
@@
 		(dnp no)
 		(fields_autoplaced yes)
-		(property "Reference" "C37"
+		(property "Reference" "C63"
 			(at 190.5 97.7899 0)
 			(effects
@@
 			(project "logix-core"
 				(path "/cf3b7c5f-6ddc-4e3f-9529-0bcf5eec6f23/ab2b6d75-2b5d-47d9-b70e-fad58fb7011e"
-					(reference "C37")
+					(reference "C63")
 					(unit 1)
 				)
@@
 		(dnp no)
 		(fields_autoplaced yes)
-		(property "Reference" "C36"
+		(property "Reference" "C61"
 			(at 212.09 50.7999 0)
 			(effects
@@
 			(project "logix-core"
 				(path "/cf3b7c5f-6ddc-4e3f-9529-0bcf5eec6f23/ab2b6d75-2b5d-47d9-b70e-fad58fb7011e"
-					(reference "C36")
+					(reference "C61")
 					(unit 1)
 				)
@@
 		(dnp no)
 		(fields_autoplaced yes)
-		(property "Reference" "#PWR016"
+		(property "Reference" "#PWR048"
 			(at 203.2 46.99 0)
 			(effects
@@
 			(project "logix-core"
 				(path "/cf3b7c5f-6ddc-4e3f-9529-0bcf5eec6f23/ab2b6d75-2b5d-47d9-b70e-fad58fb7011e"
-					(reference "#PWR016")
+					(reference "#PWR048")
 					(unit 1)
 				)
@@
 		(dnp no)
 		(fields_autoplaced yes)
-		(property "Reference" "#PWR060"
+		(property "Reference" "#PWR051"
 			(at 198.12 63.5 0)
 			(effects
@@
 			(project "logix-core"
 				(path "/cf3b7c5f-6ddc-4e3f-9529-0bcf5eec6f23/ab2b6d75-2b5d-47d9-b70e-fad58fb7011e"
-					(reference "#PWR060")
+					(reference "#PWR051")
 					(unit 1)
 				)
@@
 		(dnp no)
 		(fields_autoplaced yes)
-		(property "Reference" "R19"
+		(property "Reference" "R17"
 			(at 177.8 87.6299 0)
 			(effects
@@
 			(project "logix-core"
 				(path "/cf3b7c5f-6ddc-4e3f-9529-0bcf5eec6f23/ab2b6d75-2b5d-47d9-b70e-fad58fb7011e"
-					(reference "R19")
+					(reference "R17")
 					(unit 1)
 				)
@@
 		(dnp no)
 		(fields_autoplaced yes)
-		(property "Reference" "R20"
+		(property "Reference" "R18"
 			(at 177.8 97.7899 0)
 			(effects
@@
 			(project "logix-core"
 				(path "/cf3b7c5f-6ddc-4e3f-9529-0bcf5eec6f23/ab2b6d75-2b5d-47d9-b70e-fad58fb7011e"
-					(reference "R20")
+					(reference "R18")
 					(unit 1)
 				)
@@
 		(dnp no)
 		(fields_autoplaced yes)
-		(property "Reference" "#PWR07"
+		(property "Reference" "#PWR058"
 			(at 73.66 165.1 0)
 			(effects
@@
 			(project "logix-core"
 				(path "/cf3b7c5f-6ddc-4e3f-9529-0bcf5eec6f23/ab2b6d75-2b5d-47d9-b70e-fad58fb7011e"
-					(reference "#PWR07")
+					(reference "#PWR058")
 					(unit 1)
 				)
@@
 		(dnp no)
 		(fields_autoplaced yes)
-		(property "Reference" "C39"
+		(property "Reference" "C62"
 			(at 212.09 87.6299 0)
 			(effects
@@
 			(project "logix-core"
 				(path "/cf3b7c5f-6ddc-4e3f-9529-0bcf5eec6f23/ab2b6d75-2b5d-47d9-b70e-fad58fb7011e"
-					(reference "C39")
+					(reference "C62")
 					(unit 1)
 				)
@@
 		(dnp no)
 		(fields_autoplaced yes)
-		(property "Reference" "U8"
+		(property "Reference" "U6"
 			(at 250.19 20.32 0)
 			(effects
@@
 			(project "logix-core"
 				(path "/cf3b7c5f-6ddc-4e3f-9529-0bcf5eec6f23/ab2b6d75-2b5d-47d9-b70e-fad58fb7011e"
-					(reference "U8")
+					(reference "U6")
 					(unit 2)
 				)
@@
 		(dnp no)
 		(fields_autoplaced yes)
-		(property "Reference" "C42"
+		(property "Reference" "C58"
 			(at 181.61 50.7999 0)
 			(effects
@@
 			(project "logix-core"
 				(path "/cf3b7c5f-6ddc-4e3f-9529-0bcf5eec6f23/ab2b6d75-2b5d-47d9-b70e-fad58fb7011e"
-					(reference "C42")
-					(unit 1)
-				)
+					(reference "C58")
+					(unit 1)
+				)

Commit message: did alot of stuff
Parts:
- C58, C59, C60, C61, C63: LCSC (none) -> C52923
- C62, C64: LCSC (none) -> C15195
- R17, R18: LCSC (none) -> C11702
- R19: LCSC (none) -> C114755
- U6: LCSC (none) -> C2803004
Changed lines of the file:
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@@
+		(polyline
+			(pts
+				(xy 137.16 45.72) (xy 137.16 67.31) (xy 144.78 67.31) (xy 144.78 45.72)
+			)
+			(stroke
+				(width 0)
+				(type dash)
+			)
+			(fill
+				(type none)
+			)
+		)
+	)
+	(rule_area
 		(polyline
 			(pts
 				(xy 137.16 69.85) (xy 137.16 88.9) (xy 144.78 88.9) (xy 144.78 69.85)
+			)
+			(stroke
+				(width 0)
+				(type dash)
+			)
+			(fill
+				(type none)
+			)
+		)
+	)
+	(rule_area
+		(polyline
+			(pts
+				(xy 82.55 116.84) (xy 82.55 129.54) (xy 87.63 129.54) (xy 87.63 116.84)
 			)
 			(stroke
@@
 			(pts
 				(xy 82.55 45.72) (xy 82.55 58.42) (xy 86.36 58.42) (xy 86.36 45.72)
-			)
-			(stroke
-				(width 0)
-				(type dash)
-			)
-			(fill
-				(type none)
-			)
-		)
-	)
-	(rule_area
-		(polyline
-			(pts
-				(xy 82.55 116.84) (xy 82.55 129.54) (xy 87.63 129.54) (xy 87.63 116.84)
-			)
-			(stroke
-				(width 0)
-				(type dash)
-			)
-			(fill
-				(type none)
-			)
-		)
-	)
-	(rule_area
-		(polyline
-			(pts
-				(xy 137.16 45.72) (xy 137.16 67.31) (xy 144.78 67.31) (xy 144.78 45.72)
 			)
 			(stroke
@@
 			)
 		)
+		(property "LCSC" "C114755"
+			(at 73.66 153.67 0)
+			(effects
+				(font
+					(size 1.27 1.27)
+				)
+			)
+		)
 		(pin "1"
 		)
@@
 			)
 		)
+		(property "LCSC" "C52923"
+			(at 198.12 52.07 0)
+			(effects
+				(font
+					(size 1.27 1.27)
+				)
+			)
+		)
 		(pin "2"
 		)
@@
 			)
 		)
+		(property "LCSC" "C2803004"
+			(at 88.9 46.99 0)
+			(effects
+				(font
+					(size 1.27 1.27)
+				)
+			)
+		)
 		(pin "R8"
 		)
@@
 			)
 		)
+		(property "LCSC" "C15195"
+			(at 198.12 99.06 0)
+			(effects
+				(font
+					(size 1.27 1.27)
+				)
+			)
+		)
 		(pin "2"
 		)
@@
 			)
 		)
+		(property "LCSC" "C52923"
+			(at 187.96 52.07 0)
+			(effects
+				(font
+					(size 1.27 1.27)
+				)
+			)
+		)
 		(pin "2"
 		)
@@
 			)
 		)
+		(property "LCSC" "C52923"
+			(at 186.69 99.06 0)
+			(effects
+				(font
+					(size 1.27 1.27)
+				)
+			)
+		)
 		(pin "2"
 		)
@@
 			)
 		)
+		(property "LCSC" "C52923"
+			(at 208.28 52.07 0)
+			(effects
+				(font
+					(size 1.27 1.27)
+				)
+			)
+		)
 		(pin "2"
 		)
@@
 			)
 		)
+		(property "LCSC" "C11702"
+			(at 175.26 88.9 0)
+			(effects
+				(font
+					(size 1.27 1.27)
+				)
+			)
+		)
 		(pin "1"
 		)
@@
 			)
 		)
+		(property "LCSC" "C11702"
+			(at 175.26 99.06 0)
+			(effects
+				(font
+					(size 1.27 1.27)
+				)
+			)
+		)
 		(pin "1"
 		)
@@
 			)
 		)
+		(property "LCSC" "C15195"
+			(at 208.28 88.9 0)
+			(effects
+				(font
+					(size 1.27 1.27)
+				)
+			)
+		)
 		(pin "2"
 		)
@@
 			)
 		)
+		(property "LCSC" "C2803004"
+			(at 227.33 30.48 0)
+			(effects
+				(font
+					(size 1.27 1.27)
+				)
+			)
+		)
 		(pin "R8"
 		)
@@
 			)
 		)
+		(property "LCSC" "C52923"
+			(at 177.8 52.07 0)
+			(effects
+				(font
+					(size 1.27 1.27)
+				)
+			)
+		)
